File: zynq7000.kicad_pcb (KiCad board)
At the start: 6 copper layers, 85.6 x 54 mm, 332 parts, among them IC1 MMPF0100NPAEP, J1 FPC 40 pins P0.5mm, J10 USB_C_Receptacle_USB2.0_16P, J11 Micro_SD_Card_Det1, J12 HDMI_A_1.4, J13 USB_C_Receptacle_USB2.0_16P, J2 FPC 40 pins P0.5mm, J3 Header 2.54mm, J4 Header 2.54mm, J5 AudioJack4, J6 Header 2.54mm, J7 USB_C_Receptacle_USB2.0_16P, J8 MX_1.25mm, J9 HR911130A, Q1 2N7002, Q2 2N7002, Q3 2N7002, SW1 SW_Push, SW2 SW_Push, SW3 SW_Push, U1 XC7Z010-1CLG400C, U10 AT93C46-10SU-2.7-T, U2 H5TC2G83EFR-xxA, U3 H5TC2G83EFR-xxA, U4 SGTL5000XNLA3, U5 BQ25601, U6 RTL8211F-CG, U7 USB3320C-EZK-TR, U8 W25Q128JVS, U9 FT4232H, X1 ASE-40MHz, Y1 25MHz, Y2 12MHz

Commit message: add overview
Parts:
- moved C152 0.40 mm to (132.9, 47.8)
- moved R82 0.40 mm to (131.9, 47.8)
- moved R85 0.37 mm to (130.9, 47.8)
- moved R50 0.29 mm to (130.6, 66.4)
- moved R51 0.23 mm to (130.6, 67.5)
- moved C153 0.23 mm to (127.9, 47.8)
- renumbered C9 to C10, C10 to C11, C11 to C12, C12 to C13, C13 to C14, C14 to C15, C15 to C16, C16 to C17, C44 to C172, C17 to C18, C18 to C19, C19 to C20, C20 to C21, C21 to C22, C22 to C23, C23 to C24, C24 to C25, C25 to C26, C26 to C27, C27 to C28, C28 to C29, C29 to C30, C30 to C31, C31 to C32, C32 to C33, C33 to C34, C34 to C35, C35 to C36, C36 to C37, C37 to C38, C38 to C39, C39 to C40, C40 to C41, C41 to C42, C42 to C43, C43 to C44, J11 to J10, J13 to J11, J4 to J13, J5 to J4, J6 to J5, J7 to J6, J8 to J7, J9 to J8, J10 to J9, R99 to R100, R41 to R101, R42 to R102, R44 to R103, R45 to R104, R46 to R105, R49 to R106, R51 to R107, R36 to R108, R37 to R36, R38 to R37, R39 to R38, R40 to R39, R43 to R40, R47 to R41, R48 to R42, R50 to R43, R52 to R44, R53 to R45, R54 to R46, R55 to R47, R56 to R48, R57 to R49, R58 to R50, R59 to R51, R60 to R52, R61 to R53, R62 to R54, R63 to R55, R64 to R56, R65 to R57, R66 to R58, R67 to R59, R68 to R60, R69 to R61, R70 to R62, R71 to R63, R72 to R64, R73 to R65, R74 to R66, R75 to R67, R76 to R68, R77 to R69, R78 to R70, R79 to R71, R80 to R72, R81 to R73, R82 to R74, R83 to R75, R84 to R76, R85 to R77, R86 to R78, R87 to R79, R88 to R80, R89 to R81, R90 to R82, R91 to R83, R92 to R84, R93 to R85, R94 to R86, R100 to R87, R101 to R88, R102 to R89, R103 to R90, R104 to R91, R105 to R92, R106 to R93, R107 to R94, R108 to R95, R95 to R96, R96 to R97, R97 to R98, R98 to R99
Connections:
- net /DRAM DDR3/DRAM_A0 renamed DRAM_A0
- net /DRAM DDR3/DRAM_A1 renamed DRAM_A1
- net /DRAM DDR3/DRAM_A10 renamed DRAM_A10
- net /DRAM DDR3/DRAM_A11 renamed DRAM_A11
- net /DRAM DDR3/DRAM_A12 renamed DRAM_A12
- net /DRAM DDR3/DRAM_A13 renamed DRAM_A13
- net /DRAM DDR3/DRAM_A14 renamed DRAM_A14
- net /DRAM DDR3/DRAM_A2 renamed DRAM_A2
- net /DRAM DDR3/DRAM_A3 renamed DRAM_A3
- net /DRAM DDR3/DRAM_A4 renamed DRAM_A4
- net /DRAM DDR3/DRAM_A5 renamed DRAM_A5
- net /DRAM DDR3/DRAM_A6 renamed DRAM_A6
- net /DRAM DDR3/DRAM_A7 renamed DRAM_A7
- net /DRAM DDR3/DRAM_A8 renamed DRAM_A8
- net /DRAM DDR3/DRAM_A9 renamed DRAM_A9
- net /DRAM DDR3/DRAM_BA0 renamed DRAM_BA0
- net /DRAM DDR3/DRAM_BA1 renamed DRAM_BA1
- net /DRAM DDR3/DRAM_BA2 renamed DRAM_BA2
- net /DRAM DDR3/DRAM_CASN renamed DRAM_CASN
- net /DRAM DDR3/DRAM_CKE renamed DRAM_CKE
- net /DRAM DDR3/DRAM_CLK_N renamed DRAM_CLK_N
- net /DRAM DDR3/DRAM_CLK_P renamed DRAM_CLK_P
- net /DRAM DDR3/DRAM_CSN renamed DRAM_CSN
- net /DRAM DDR3/DRAM_DM0 renamed DRAM_DM0
- net /DRAM DDR3/DRAM_DM1 renamed DRAM_DM1
- net /DRAM DDR3/DRAM_DQ0 renamed DRAM_DQ0
- net /DRAM DDR3/DRAM_DQ1 renamed DRAM_DQ1
- net /DRAM DDR3/DRAM_DQ10 renamed DRAM_DQ10
- net /DRAM DDR3/DRAM_DQ11 renamed DRAM_DQ11
- net /DRAM DDR3/DRAM_DQ12 renamed DRAM_DQ12
- net /DRAM DDR3/DRAM_DQ13 renamed DRAM_DQ13
- net /DRAM DDR3/DRAM_DQ14 renamed DRAM_DQ14
- net /DRAM DDR3/DRAM_DQ15 renamed DRAM_DQ15
- net /DRAM DDR3/DRAM_DQ2 renamed DRAM_DQ2
- net /DRAM DDR3/DRAM_DQ3 renamed DRAM_DQ3
- net /DRAM DDR3/DRAM_DQ4 renamed DRAM_DQ4
- net /DRAM DDR3/DRAM_DQ5 renamed DRAM_DQ5
- net /DRAM DDR3/DRAM_DQ6 renamed DRAM_DQ6
- net /DRAM DDR3/DRAM_DQ7 renamed DRAM_DQ7
- net /DRAM DDR3/DRAM_DQ8 renamed DRAM_DQ8
- net /DRAM DDR3/DRAM_DQ9 renamed DRAM_DQ9
- net /DRAM DDR3/DRAM_DQS0_N renamed DRAM_DQS0_N
- net /DRAM DDR3/DRAM_DQS0_P renamed DRAM_DQS0_P
- net /DRAM DDR3/DRAM_DQS1_N renamed DRAM_DQS1_N
- net /DRAM DDR3/DRAM_DQS1_P renamed DRAM_DQS1_P
- net /DRAM DDR3/DRAM_ODT renamed DRAM_ODT
- net /DRAM DDR3/DRAM_RASN renamed DRAM_RASN
- net /DRAM DDR3/DRAM_RSTN renamed DRAM_RSTN
- net /DRAM DDR3/DRAM_WEN renamed DRAM_WEN
Routing:
- net /Bank 34 (3.3V)/FPGA_IO34_L1N: track 14.1 -> 14.9 mm
- net /PL Configuration/FPGA_PL_INIT_B: track 46.0 -> 46.8 mm
- net /Gigabit Ethernet PHY/ETH_XTAL_IN: track 7.33 -> 6.78 mm
