File: zynq7000.kicad_pcb (KiCad board)
At the start: 6 copper layers, 85.6 x 54 mm, 332 parts, among them IC1 MMPF0100NPAEP, J1 FPC 40 pins P0.5mm, J10 Micro_SD_Card_Det1, J11 USB_C_Receptacle_USB2.0_16P, J12 HDMI_A_1.4, J13 Header 2.54mm, J2 FPC 40 pins P0.5mm, J3 Header 2.54mm, J4 AudioJack4, J5 Header 2.54mm, J6 USB_C_Receptacle_USB2.0_16P, J7 MX_1.25mm, J8 HR911130A, J9 USB_C_Receptacle_USB2.0_16P, Q1 2N7002, Q2 2N7002, Q3 2N7002, SW1 SW_Push, SW2 SW_Push, SW3 SW_Push, U1 XC7Z010-1CLG400C, U10 AT93C46-10SU-2.7-T, U2 H5TC2G83EFR-xxA, U3 H5TC2G83EFR-xxA, U4 SGTL5000XNLA3, U5 BQ25601, U6 RTL8211F-CG, U7 USB3320C-EZK-TR, U8 W25Q128JVS, U9 FT4232H, X1 ASE-40MHz, Y1 25MHz, Y2 12MHz

Commit message: update
Parts:
- added C174: 4u7, Capacitor_SMD:C_0402_1005Metric, F.Cu at (114.9, 90.7)
- added C175: 1u, Capacitor_SMD:C_0402_1005Metric, F.Cu at (114.9, 88.8)
- added R109: 1k2, Resistor_SMD:R_0402_1005Metric, F.Cu at (133.9, 47.8)
- added R110: 10k, Resistor_SMD:R_0402_1005Metric, F.Cu at (146.9, 72.1)
- C1, C10, C100, C103, C106, C109, C11, C112, C115, C119, C12, C120, C121, C122, C124, C126, C127, C128, C129, C13, C133, C134, C135, C136, C14, C143, C15, C16, C17, C172, C18, C19, C2, C20, C21, C22, C23, C24, C25, C26, C3, C4, C5, C6, C7, C8, C81, C94, C95, C96, C99: value 470n -> 1u
- C151: value 2u2 -> 4u7
- C27, C28, C47: value 10n -> 100n
- C59, C60, C61, C62, C63, C64, C65: value 4u7 -> 10u
- C79, C85: value 1u -> 4u7
- C87: footprint Capacitor_SMD:C_0402_1005Metric -> Capacitor_SMD:C_0603_1608Metric
- D5: value STAT -> BLUE
- D6: value PG -> GREEN
- J4: value AudioJack4 -> PJ320D
- R2, R5: value 90R -> 120R
- R3, R4: value 270R -> 240R
- R78: value 2k49 -> 3k3
- R85: value 8k06 -> 6k8
- U5: footprint Package_DFN_QFN:Texas_RTW_WQFN-24-1EP_4x4mm_P0.5mm_EP2.7x2.7mm_ThermalVias -> Custom:WQFN-24-1EP_4x4mm_P0.5mm_BQ25601
- U6: footprint Custom:RTL8211F-CG_RTK -> Custom:QFN_40_7x7mm_RTL8211F
- U7: footprint Custom:QFN32_5X5MC_MCH -> Custom:QFN32_5X5_USB3320
- X1: value ASE-40MHz -> 40MHz
- moved C138 1.83 mm to (146.9, 74.0)
- moved R102 0.71 mm to (106.0, 49.0), turned to -90 degrees
- moved C87 0.34 mm to (95.8, 88.1)
- moved L6 0.27 mm to (92.9, 89.7)
- moved RN1 0.19 mm to (139.4, 56.2)
Connections:
- C50 pad 1: +1V8 -> +1V8A
- IC1 pad 28: unconnected-(IC1-VGEN4-Pad28) -> +1V8A
- R85 pad 2: GND -> Net-(R109-Pad1)
- R94 pad 2: /FTDI/FTDI_EEPROM_DATA -> Net-(U10-DO)
- R95 pad 1: /FTDI/FTDI_EEPROM_DATA -> Net-(U10-DO)
- R95 pad 2: Net-(U10-DI) -> /FTDI/FTDI_EEPROM_DATA
- U1 pad D9: SDIO1_D0 -> SDIO1_CLK
- U1 pad E9: SDIO1_CLK -> SDIO1_D0
- U10 pad 5: Net-(U10-DI) -> /FTDI/FTDI_EEPROM_DATA
- U10 pad 6: /FTDI/FTDI_EEPROM_DATA -> Net-(U10-DO)
- U4 pad 3: +1V8 -> +1V8A
- U9 pad 21: unconnected-(U9-ADBUS4-Pad21) -> +3V3
Routing:
- net +1V8A: track 0.00 -> 51.5 mm, vias 0 -> 4
- net Net-(U10-DO): track 0.00 -> 10.3 mm
- net /FTDI/FTDI_EEPROM_DATA: track 17.2 -> 13.6 mm
- net Net-(R109-Pad1): track 0.00 -> 3.42 mm, vias 0 -> 2
- net Net-(U10-DI): track 2.35 -> 0.00 mm
- net Net-(U6A-RSET): track 2.93 -> 5.02 mm
- net Net-(U5-REGN): track 8.26 -> 10.2 mm
- net SDIO1_CD: track 57.4 -> 55.9 mm
- net /Gigabit Ethernet PHY/ETH_RXD3_R: track 8.75 -> 10.2 mm
- net /Gigabit Ethernet PHY/ETH_RXCTL_R: track 12.6 -> 13.9 mm
- net QSPI0_CSN: track 20.9 -> 22.1 mm
- net +1V8: track 41.8 -> 40.7 mm, vias 79 -> 78
- net Net-(U5-~{PG}): track 14.2 -> 15.3 mm
- net +1V0: track 17.1 -> 18.1 mm
- net QSPI0_D2: track 22.2 -> 23.2 mm
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Other:
- board text added: "B"
- board text added: "T"
- board text added: "design by yusenpai"
