File: bms.kicad_sch (KiCad schematic)
At the start: 20 parts, among them J7 USB_C_Receptacle_USB2.0_16P, J8 MX_1.25mm, U5 BQ25601

Commit message: add overview
Parts:
- renumbered J7 to J6, J8 to J7, R69 to R61, R70 to R62, R71 to R63, R72 to R64, R73 to R65, R74 to R66, R75 to R67
Other:
- note added: "BMS"
- note removed: "Charger"
Changed lines of the file:
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@@
 		)
 	)
-	(text "Charger"
+	(text "BMS"
 		(exclude_from_sim no)
 		(at 63.5 49.53 0)
@@
 				)
 				(justify right)
-				(hide yes)
 			)
 		)
@@
 				)
 				(justify right)
-				(hide yes)
 			)
 		)
@@
 				)
 				(justify right)
-				(hide yes)
 			)
 		)
@@
 		(dnp no)
 		(fields_autoplaced yes)
-		(property "Reference" "#PWR0116"
+		(property "Reference" "#PWR0110"
 			(at 138.43 80.01 0)
 			(effects
@@
 			(project "zynq7000"
 				(path "/b3b2a4a2-12d8-4419-9374-817f22e1ad00/70bcdf00-8a72-4540-b7e3-7a221388cfd4"
-					(reference "#PWR0116")
+					(reference "#PWR0110")
 					(unit 1)
 				)
@@
 		(dnp no)
 		(fields_autoplaced yes)
-		(property "Reference" "#PWR0127"
+		(property "Reference" "#PWR0121"
 			(at 176.53 123.19 0)
 			(effects
@@
 			(project "zynq7000"
 				(path "/b3b2a4a2-12d8-4419-9374-817f22e1ad00/70bcdf00-8a72-4540-b7e3-7a221388cfd4"
-					(reference "#PWR0127")
+					(reference "#PWR0121")
 					(unit 1)
 				)
@@
 		(on_board yes)
 		(dnp no)
-		(property "Reference" "R75"
+		(property "Reference" "R67"
 			(at 178.054 111.76 0)
 			(effects
@@
 			(project "zynq7000"
 				(path "/b3b2a4a2-12d8-4419-9374-817f22e1ad00/70bcdf00-8a72-4540-b7e3-7a221388cfd4"
-					(reference "R75")
+					(reference "R67")
 					(unit 1)
 				)
@@
 		(on_board yes)
 		(dnp no)
-		(property "Reference" "R72"
+		(property "Reference" "R64"
 			(at 179.07 82.296 90)
 			(effects
@@
 			(project "zynq7000"
 				(path "/b3b2a4a2-12d8-4419-9374-817f22e1ad00/70bcdf00-8a72-4540-b7e3-7a221388cfd4"
-					(reference "R72")
+					(reference "R64")
 					(unit 1)
 				)
@@
 		(on_board yes)
 		(dnp no)
-		(property "Reference" "J7"
+		(property "Reference" "J6"
 			(at 96.52 62.23 0)
 			(effects
@@
 			(project "zynq7000"
 				(path "/b3b2a4a2-12d8-4419-9374-817f22e1ad00/70bcdf00-8a72-4540-b7e3-7a221388cfd4"
-					(reference "J7")
+					(reference "J6")
 					(unit 1)
 				)
@@
 		(on_board yes)
 		(dnp no)
-		(property "Reference" "R74"
+		(property "Reference" "R66"
 			(at 178.054 102.87 0)
 			(effects
@@
 			(project "zynq7000"
 				(path "/b3b2a4a2-12d8-4419-9374-817f22e1ad00/70bcdf00-8a72-4540-b7e3-7a221388cfd4"
-					(reference "R74")
+					(reference "R66")
 					(unit 1)
 				)
@@
 		(on_board yes)
 		(dnp no)
-		(property "Reference" "R73"
+		(property "Reference" "R65"
 			(at 179.07 90.932 90)
 			(effects
@@
 			(project "zynq7000"
 				(path "/b3b2a4a2-12d8-4419-9374-817f22e1ad00/70bcdf00-8a72-4540-b7e3-7a221388cfd4"
-					(reference "R73")
+					(reference "R65")
 					(unit 1)
 				)
@@
 		(on_board yes)
 		(dnp no)
-		(property "Reference" "#PWR0113"
+		(property "Reference" "#PWR0107"
 			(at 106.68 67.31 0)
 			(effects
@@
 			(project "zynq7000"
 				(path "/b3b2a4a2-12d8-4419-9374-817f22e1ad00/70bcdf00-8a72-4540-b7e3-7a221388cfd4"
-					(reference "#PWR0113")
+					(reference "#PWR0107")
 					(unit 1)
 				)
@@
 		(on_board yes)
 		(dnp no)
-		(property "Reference" "J8"
+		(property "Reference" "J7"
 			(at 228.6 90.17 0)
 			(effects
@@
 			(project "zynq7000"
 				(path "/b3b2a4a2-12d8-4419-9374-817f22e1ad00/70bcdf00-8a72-4540-b7e3-7a221388cfd4"
-					(reference "J8")
+					(reference "J7")
 					(unit 1)
 				)
@@
 		(dnp yes)
 		(fields_autoplaced yes)
-		(property "Reference" "R71"
+		(property "Reference" "R63"
 			(at 109.22 81.28 0)
 			(effects
@@
 			(project "zynq7000"
 				(path "/b3b2a4a2-12d8-4419-9374-817f22e1ad00/70bcdf00-8a72-4540-b7e3-7a221388cfd4"
-					(reference "R71")
+					(reference "R63")
 					(unit 1)
 				)
@@
 		(on_board yes)
 		(dnp no)
-		(property "Reference" "#PWR0119"
+		(property "Reference" "#PWR0113"
 			(at 200.66 96.52 0)
 			(effects
@@
 			(project "zynq7000"
 				(path "/b3b2a4a2-12d8-4419-9374-817f22e1ad00/70bcdf00-8a72-4540-b7e3-7a221388cfd4"
-					(reference "#PWR0119")
+					(reference "#PWR0113")
 					(unit 1)
 				)
@@
 		(dnp no)
 		(fields_autoplaced yes)
-		(property "Reference" "#PWR0123"
+		(property "Reference" "#PWR0117"
 			(at 198.12 113.03 0)
 			(effects
@@
 			(project "zynq7000"
 				(path "/b3b2a4a2-12d8-4419-9374-817f22e1ad00/70bcdf00-8a72-4540-b7e3-7a221388cfd4"
-					(reference "#PWR0123")
+					(reference "#PWR0117")
 					(unit 1)
 				)
@@
 		(dnp no)
 		(fields_autoplaced yes)
-		(property "Reference" "#PWR0126"
+		(property "Reference" "#PWR0120"
 			(at 161.29 123.19 0)
 			(effects
@@
 			(project "zynq7000"
 				(path "/b3b2a4a2-12d8-4419-9374-817f22e1ad00/70bcdf00-8a72-4540-b7e3-7a221388cfd4"
-					(reference "#PWR0126")
+					(reference "#PWR0120")
 					(unit 1)
 				)
@@
 		(on_board yes)
 		(dnp no)
-		(property "Reference" "#PWR0114"
+		(property "Reference" "#PWR0108"
 			(at 193.04 68.58 0)
 			(effects
@@
 			(project "zynq7000"
 				(path "/b3b2a4a2-12d8-4419-9374-817f22e1ad00/70bcdf00-8a72-4540-b7e3-7a221388cfd4"
-					(reference "#PWR0114")
+					(reference "#PWR0108")
 					(unit 1)
 				)
@@
 		(dnp no)
 		(fields_autoplaced yes)
-		(property "Reference" "#PWR0125"
+		(property "Reference" "#PWR0119"
 			(at 135.89 123.19 0)
 			(effects
@@
 			(project "zynq7000"
 				(path "/b3b2a4a2-12d8-4419-9374-817f22e1ad00/70bcdf00-8a72-4540-b7e3-7a221388cfd4"
-					(reference "#PWR0125")
+					(reference "#PWR0119")
 					(unit 1)
 				)
@@
 		(dnp no)
 		(fields_autoplaced yes)
-		(property "Reference" "#PWR0121"
+		(property "Reference" "#PWR0115"
 			(at 78.74 113.03 0)
 			(effects
@@
 			(project "zynq7000"
 				(path "/b3b2a4a2-12d8-4419-9374-817f22e1ad00/70bcdf00-8a72-4540-b7e3-7a221388cfd4"
-					(reference "#PWR0121")
+					(reference "#PWR0115")
 					(unit 1)
 				)
@@
 		(dnp no)
 		(fields_autoplaced yes)
-		(property "Reference" "#PWR0117"
+		(property "Reference" "#PWR0111"
 			(at 190.5 80.01 0)
 			(effects
@@
 			(project "zynq7000"
 				(path "/b3b2a4a2-12d8-4419-9374-817f22e1ad00/70bcdf00-8a72-4540-b7e3-7a221388cfd4"
-					(reference "#PWR0117")
+					(reference "#PWR0111")
 					(unit 1)
 				)
@@
 		(dnp no)
 		(fields_autoplaced yes)
-		(property "Reference" "#PWR0120"
+		(property "Reference" "#PWR0114"
 			(at 142.24 105.41 0)
 			(effects
@@
 			(project "zynq7000"
 				(path "/b3b2a4a2-12d8-4419-9374-817f22e1ad00/70bcdf00-8a72-4540-b7e3-7a221388cfd4"
-					(reference "#PWR0120")
+					(reference "#PWR0114")
 					(unit 1)
 				)
@@
 		(dnp no)
 		(fields_autoplaced yes)
-		(property "Reference" "#PWR0124"
+		(property "Reference" "#PWR0118"
 			(at 220.98 121.92 0)
 			(effects
@@
 			(project "zynq7000"
 				(path "/b3b2a4a2-12d8-4419-9374-817f22e1ad00/70bcdf00-8a72-4540-b7e3-7a221388cfd4"
-					(reference "#PWR0124")
+					(reference "#PWR0118")
 					(unit 1)
 				)
@@
 		(on_board yes)
 		(dnp no)
-		(property "Reference" "#PWR0118"
+		(property "Reference" "#PWR0112"
 			(at 193.04 88.9 0)
 			(effects
@@
 			(project "zynq7000"
 				(path "/b3b2a4a2-12d8-4419-9374-817f22e1ad00/70bcdf00-8a72-4540-b7e3-7a221388cfd4"
-					(reference "#PWR0118")
+					(reference "#PWR0112")
 					(unit 1)
 				)
@@
 		(dnp no)
 		(fields_autoplaced yes)
-		(property "Reference" "#PWR0122"
+		(property "Reference" "#PWR0116"
 			(at 187.96 113.03 0)
 			(effects
@@
 			(project "zynq7000"
 				(path "/b3b2a4a2-12d8-4419-9374-817f22e1ad00/70bcdf00-8a72-4540-b7e3-7a221388cfd4"
-					(reference "#PWR0122")
+					(reference "#PWR0116")
 					(unit 1)
 				)
@@
 		(on_board yes)
 		(dnp no)
-		(property "Reference" "R69"
+		(property "Reference" "R61"
 			(at 107.95 68.58 90)
 			(effects
@@
 			(project "zynq7000"
 				(path "/b3b2a4a2-12d8-4419-9374-817f22e1ad00/70bcdf00-8a72-4540-b7e3-7a221388cfd4"
-					(reference "R69")
+					(reference "R61")
 					(unit 1)
 				)
@@
 		(on_board yes)
 		(dnp no)
-		(property "Reference" "R70"
+		(property "Reference" "R62"
 			(at 107.95 76.2 90)
 			(effects
@@
 			(project "zynq7000"
 				(path "/b3b2a4a2-12d8-4419-9374-817f22e1ad00/70bcdf00-8a72-4540-b7e3-7a221388cfd4"
-					(reference "R70")
+					(reference "R62")
 					(unit 1)
 				)
@@
 		(dnp no)
 		(fields_autoplaced yes)
-		(property "Reference" "#PWR0115"
+		(property "Reference" "#PWR0109"
 			(at 114.3 80.01 0)
 			(effects
@@
 			(project "zynq7000"
 				(path "/b3b2a4a2-12d8-4419-9374-817f22e1ad00/70bcdf00-8a72-4540-b7e3-7a221388cfd4"
-					(reference "#PWR0115")
+					(reference "#PWR0109")
 					(unit 1)
 				)

Commit message: update
Parts:
- C85: value 1u -> 4u7
- C87: footprint Capacitor_SMD:C_0402_1005Metric -> Capacitor_SMD:C_0603_1608Metric
- D5: value STAT -> BLUE
- D6: value PG -> GREEN
- U5: footprint Package_DFN_QFN:Texas_RTW_WQFN-24-1EP_4x4mm_P0.5mm_EP2.7x2.7mm_ThermalVias -> Custom:WQFN-24-1EP_4x4mm_P0.5mm_BQ25601
Changed lines of the file:
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@@
 				)
 				(justify right)
+				(hide yes)
 			)
 		)
@@
 				)
 				(justify right)
+				(hide yes)
 			)
 		)
@@
 				)
 				(justify right)
+				(hide yes)
 			)
 		)
@@
 			)
 		)
-		(property "Footprint" "Package_DFN_QFN:Texas_RTW_WQFN-24-1EP_4x4mm_P0.5mm_EP2.7x2.7mm_ThermalVias"
+		(property "Footprint" "Custom:WQFN-24-1EP_4x4mm_P0.5mm_BQ25601"
 			(at 161.29 59.69 0)
 			(effects
@@
 			)
 		)
-		(property "Footprint" "Capacitor_SMD:C_0402_1005Metric"
+		(property "Footprint" "Capacitor_SMD:C_0603_1608Metric"
 			(at 190.5 69.85 0)
 			(effects
@@
 			)
 		)
-		(property "Value" "PG"
+		(property "Value" "GREEN"
 			(at 187.96 92.964 0)
 			(effects
@@
 			)
 		)
-		(property "Value" "1u"
+		(property "Value" "4u7"
 			(at 140.97 71.1262 0)
 			(effects
@@
 			)
 		)
-		(property "Value" "STAT"
+		(property "Value" "BLUE"
 			(at 187.96 83.312 0)
 			(effects
