File: ftdi.kicad_sch (KiCad schematic)
At the start: 29 parts, among them J13 USB_C_Receptacle_USB2.0_16P, U10 AT93C46-10SU-2.7-T, U9 FT4232H, Y2 12MHz

Commit message: add overview
Parts:
- renumbered J13 to J11, R100 to R87, R101 to R88, R102 to R89, R103 to R90, R104 to R91, R105 to R92, R106 to R93, R107 to R94, R108 to R95

Commit message: update
Connections:
- net +3V3: now also U9.21 (ADBUS4)
- net FTDI_EEPROM_DATA: now also R95.2, U10.5 (DI); no longer R94.2, R95.1, U10.6 (DO)
- new net: R94.2, R95.1, U10.6 (DO)
- no-connect marks 28 -> 27
Other:
- moved on the sheet: R95
Changed lines of the file:
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@@
+	)
+	(junction
+		(at 105.41 123.19)
+		(diameter 0)
+		(color 0 0 0 0)
 	)
 	(junction
@@
 	)
 	(junction
-		(at 105.41 125.73)
-		(diameter 0)
-		(color 0 0 0 0)
-	)
-	(junction
 		(at 187.96 154.94)
 		(diameter 0)
@@
 	)
 	(junction
-		(at 105.41 123.19)
-		(diameter 0)
-		(color 0 0 0 0)
-	)
-	(junction
 		(at 195.58 43.18)
 		(diameter 0)
@@
 	)
 	(junction
+		(at 97.79 125.73)
+		(diameter 0)
+		(color 0 0 0 0)
+	)
+	(junction
 		(at 227.33 39.37)
 		(diameter 0)
@@
 	)
 	(no_connect
-		(at 215.9 62.23)
-	)
-	(no_connect
 		(at 215.9 143.51)
 	)
@@
 	(wire
 		(pts
-			(xy 105.41 125.73) (xy 102.87 125.73)
-		)
-		(stroke
-			(width 0)
-			(type default)
-		)
-	)
-	(wire
-		(pts
 			(xy 245.11 46.99) (xy 245.11 45.72)
 		)
@@
 	(wire
 		(pts
+			(xy 96.52 123.19) (xy 105.41 123.19)
+		)
+		(stroke
+			(width 0)
+			(type default)
+		)
+	)
+	(wire
+		(pts
 			(xy 111.76 116.84) (xy 111.76 120.65)
 		)
@@
 	(wire
 		(pts
+			(xy 109.22 125.73) (xy 109.22 132.08)
+		)
+		(stroke
+			(width 0)
+			(type default)
+		)
+	)
+	(wire
+		(pts
 			(xy 81.28 100.33) (xy 81.28 101.6)
 		)
@@
 	(wire
 		(pts
-			(xy 105.41 125.73) (xy 133.35 125.73)
-		)
-		(stroke
-			(width 0)
-			(type default)
-		)
-	)
-	(wire
-		(pts
 			(xy 107.95 38.1) (xy 107.95 39.37)
 		)
@@
 	(wire
 		(pts
-			(xy 96.52 123.19) (xy 105.41 123.19)
-		)
-		(stroke
-			(width 0)
-			(type default)
-		)
-	)
-	(wire
-		(pts
 			(xy 125.73 57.15) (xy 125.73 58.42)
 		)
@@
 	(wire
 		(pts
+			(xy 97.79 125.73) (xy 99.06 125.73)
+		)
+		(stroke
+			(width 0)
+			(type default)
+		)
+	)
+	(wire
+		(pts
 			(xy 137.16 143.51) (xy 137.16 144.78)
 		)
@@
 	(wire
 		(pts
+			(xy 215.9 62.23) (xy 217.17 62.23)
+		)
+		(stroke
+			(width 0)
+			(type default)
+		)
+	)
+	(wire
+		(pts
 			(xy 140.97 140.97) (xy 154.94 140.97)
 		)
@@
 	(wire
 		(pts
+			(xy 105.41 116.84) (xy 105.41 123.19)
+		)
+		(stroke
+			(width 0)
+			(type default)
+		)
+	)
+	(wire
+		(pts
 			(xy 139.7 140.97) (xy 140.97 140.97)
 		)
@@
 	(wire
 		(pts
+			(xy 97.79 125.73) (xy 97.79 132.08)
+		)
+		(stroke
+			(width 0)
+			(type default)
+		)
+	)
+	(wire
+		(pts
 			(xy 137.16 46.99) (xy 134.62 46.99)
 		)
@@
 	(wire
 		(pts
+			(xy 105.41 123.19) (xy 105.41 125.73)
+		)
+		(stroke
+			(width 0)
+			(type default)
+		)
+	)
+	(wire
+		(pts
 			(xy 137.16 39.37) (xy 137.16 38.1)
 		)
@@
 	(wire
 		(pts
+			(xy 109.22 125.73) (xy 133.35 125.73)
+		)
+		(stroke
+			(width 0)
+			(type default)
+		)
+	)
+	(wire
+		(pts
 			(xy 96.52 80.01) (xy 154.94 80.01)
 		)
@@
 	(wire
 		(pts
-			(xy 105.41 123.19) (xy 105.41 125.73)
-		)
-		(stroke
-			(width 0)
-			(type default)
-		)
-	)
-	(wire
-		(pts
 			(xy 198.12 38.1) (xy 198.12 39.37)
 		)
@@
 	(wire
 		(pts
-			(xy 105.41 116.84) (xy 105.41 123.19)
-		)
-		(stroke
-			(width 0)
-			(type default)
-		)
-	)
-	(wire
-		(pts
 			(xy 215.9 100.33) (xy 231.14 100.33)
 		)
@@
 	(wire
 		(pts
+			(xy 104.14 125.73) (xy 105.41 125.73)
+		)
+		(stroke
+			(width 0)
+			(type default)
+		)
+	)
+	(wire
+		(pts
 			(xy 218.44 40.64) (xy 218.44 39.37)
+		)
+		(stroke
+			(width 0)
+			(type default)
+		)
+	)
+	(wire
+		(pts
+			(xy 97.79 132.08) (xy 109.22 132.08)
 		)
 		(stroke
@@
 				)
 				(justify left)
+				(hide yes)
 			)
 		)
@@
 				)
 				(justify left)
+				(hide yes)
 			)
 		)
@@
 				)
 				(justify left)
+				(hide yes)
 			)
 		)
@@
 				)
 				(justify left)
+				(hide yes)
 			)
 		)
@@
 				)
 				(justify left)
+				(hide yes)
 			)
 		)
@@
 				)
 				(justify left)
+				(hide yes)
 			)
 		)
@@
 				)
 				(justify left)
+				(hide yes)
 			)
 		)
@@
 				)
 				(justify left)
+				(hide yes)
 			)
 		)
@@
 				)
 				(justify left)
+				(hide yes)
 			)
 		)
@@
 				)
 				(justify left)
+				(hide yes)
 			)
 		)
@@
 				)
 				(justify left)
+				(hide yes)
 			)
 		)
@@
 	(symbol
 		(lib_id "Device:R_Small")
-		(at 100.33 125.73 270)
+		(at 101.6 125.73 270)
 		(unit 1)
 		(exclude_from_sim no)
@@
 		(dnp no)
 		(property "Reference" "R95"
-			(at 100.3413 127.6689 90)
+			(at 101.6113 127.6689 90)
 			(effects
 				(font
@@
 		)
 		(property "Value" "2k"
-			(at 100.33 129.54 90)
+			(at 101.6 129.54 90)
 			(effects
 				(font
@@
 		)
 		(property "Footprint" "Resistor_SMD:R_0402_1005Metric"
-			(at 100.33 125.73 0)
+			(at 101.6 125.73 0)
 			(effects
 				(font
@@
 		)
 		(property "Datasheet" "~"
-			(at 100.33 125.73 0)
+			(at 101.6 125.73 0)
 			(effects
 				(font
@@
 		)
 		(property "Description" "Resistor, small symbol"
-			(at 100.33 125.73 0)
+			(at 101.6 125.73 0)
 			(effects
 				(font
@@
 					(unit 1)
 				)
+			)
+		)
+	)
+	(symbol
+		(lib_id "power:+1V8")
+		(at 217.17 62.23 270)
+		(unit 1)
+		(exclude_from_sim no)
+		(in_bom yes)
+		(on_board yes)
+		(dnp no)
+		(property "Reference" "#PWR0241"
+			(at 213.36 62.23 0)
+			(effects
+				(font
+					(size 1.27 1.27)
+				)
+				(hide yes)
+			)
+		)
+		(property "Value" "+3V3"
+			(at 222.25 62.23 90)
+			(effects
+				(font
+					(size 1.27 1.27)
+				)
+			)
+		)
+		(property "Footprint" ""
+			(at 217.17 62.23 0)
+			(effects
+				(font
+					(size 1.27 1.27)
+				)
+				(hide yes)
+			)
+		)
+		(property "Datasheet" ""
+			(at 217.17 62.23 0)
+			(effects
+				(font
+					(size 1.27 1.27)
+				)
+				(hide yes)
+			)
+		)
+		(property "Description" "Power symbol creates a global label with name \"+1V8\""
+			(at 217.17 62.23 0)
+			(effects
+				(font
+					(size 1.27 1.27)
+				)
+				(hide yes)
+			)
+		)
+		(pin "1"
+		)
+		(instances
+			(project "zynq7000"
+				(path "/b3b2a4a2-12d8-4419-9374-817f22e1ad00/bd263c9f-3ef6-4195-a21c-f788a41402bb"
+					(reference "#PWR0241")
+					(unit 1)
+				)
