File: pl_config.kicad_sch (KiCad schematic)
At the start: 19 parts, among them J3 Header 2.54mm, SW1 SW_Push, SW2 SW_Push, U1 XC7Z010-1CLG400C

Commit message: add overview
Parts:
- renumbered R37 to R36, R38 to R37, R39 to R38, R40 to R39, R43 to R40, R47 to R41, R48 to R42, R50 to R43
Changed lines of the file:
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@@
 				)
 				(justify right)
-				(hide yes)
 			)
 		)
@@
 				)
 				(justify right)
-				(hide yes)
 			)
 		)
@@
 				)
 				(justify left)
-				(hide yes)
 			)
 		)
@@
 				)
 				(justify right)
-				(hide yes)
 			)
 		)
@@
 				)
 				(justify left)
-				(hide yes)
 			)
 		)
@@
 				)
 				(justify right)
-				(hide yes)
 			)
 		)
@@
 				)
 				(justify right)
-				(hide yes)
 			)
 		)
@@
 		(on_board yes)
 		(dnp no)
-		(property "Reference" "R48"
+		(property "Reference" "R42"
 			(at 110.49 138.43 0)
 			(effects
@@
 			(project "zynq7000"
 				(path "/b3b2a4a2-12d8-4419-9374-817f22e1ad00/b5d6f844-b9aa-4334-b3f0-dc08737c0a31"
-					(reference "R48")
+					(reference "R42")
 					(unit 1)
 				)
@@
 		(on_board yes)
 		(dnp no)
-		(property "Reference" "R50"
+		(property "Reference" "R43"
 			(at 127 141.478 90)
 			(effects
@@
 			(project "zynq7000"
 				(path "/b3b2a4a2-12d8-4419-9374-817f22e1ad00/b5d6f844-b9aa-4334-b3f0-dc08737c0a31"
-					(reference "R50")
+					(reference "R43")
 					(unit 1)
 				)
@@
 		(on_board yes)
 		(dnp no)
-		(property "Reference" "R37"
+		(property "Reference" "R36"
 			(at 74.93 57.15 0)
 			(effects
@@
 			(project "zynq7000"
 				(path "/b3b2a4a2-12d8-4419-9374-817f22e1ad00/b5d6f844-b9aa-4334-b3f0-dc08737c0a31"
-					(reference "R37")
+					(reference "R36")
 					(unit 1)
 				)
@@
 		(on_board yes)
 		(dnp no)
-		(property "Reference" "R38"
+		(property "Reference" "R37"
 			(at 81.28 57.15 0)
 			(effects
@@
 			(project "zynq7000"
 				(path "/b3b2a4a2-12d8-4419-9374-817f22e1ad00/b5d6f844-b9aa-4334-b3f0-dc08737c0a31"
-					(reference "R38")
+					(reference "R37")
 					(unit 1)
 				)
@@
 		(dnp no)
 		(fields_autoplaced yes)
-		(property "Reference" "#PWR053"
+		(property "Reference" "#PWR049"
 			(at 132.08 137.16 0)
 			(effects
@@
 			(project "zynq7000"
 				(path "/b3b2a4a2-12d8-4419-9374-817f22e1ad00/b5d6f844-b9aa-4334-b3f0-dc08737c0a31"
-					(reference "#PWR053")
+					(reference "#PWR049")
 					(unit 1)
 				)
@@
 		(on_board yes)
 		(dnp no)
-		(property "Reference" "R40"
+		(property "Reference" "R39"
 			(at 110.49 111.76 0)
 			(effects
@@
 			(project "zynq7000"
 				(path "/b3b2a4a2-12d8-4419-9374-817f22e1ad00/b5d6f844-b9aa-4334-b3f0-dc08737c0a31"
-					(reference "R40")
+					(reference "R39")
 					(unit 1)
 				)
@@
 		(on_board yes)
 		(dnp no)
-		(property "Reference" "#PWR050"
+		(property "Reference" "#PWR047"
 			(at 132.08 120.65 0)
 			(effects
@@
 			(project "zynq7000"
 				(path "/b3b2a4a2-12d8-4419-9374-817f22e1ad00/b5d6f844-b9aa-4334-b3f0-dc08737c0a31"
-					(reference "#PWR050")
+					(reference "#PWR047")
 					(unit 1)
 				)
@@
 		(on_board yes)
 		(dnp no)
-		(property "Reference" "#PWR048"
+		(property "Reference" "#PWR046"
 			(at 111.76 113.03 0)
 			(effects
@@
 			(project "zynq7000"
 				(path "/b3b2a4a2-12d8-4419-9374-817f22e1ad00/b5d6f844-b9aa-4334-b3f0-dc08737c0a31"
-					(reference "#PWR048")
+					(reference "#PWR046")
 					(unit 1)
 				)
@@
 		(on_board yes)
 		(dnp no)
-		(property "Reference" "#PWR042"
+		(property "Reference" "#PWR041"
 			(at 154.94 41.91 0)
 			(effects
@@
 			(project "zynq7000"
 				(path "/b3b2a4a2-12d8-4419-9374-817f22e1ad00/b5d6f844-b9aa-4334-b3f0-dc08737c0a31"
-					(reference "#PWR042")
+					(reference "#PWR041")
 					(unit 1)
 				)
@@
 		(on_board yes)
 		(dnp no)
-		(property "Reference" "#PWR054"
+		(property "Reference" "#PWR050"
 			(at 111.76 139.7 0)
 			(effects
@@
 			(project "zynq7000"
 				(path "/b3b2a4a2-12d8-4419-9374-817f22e1ad00/b5d6f844-b9aa-4334-b3f0-dc08737c0a31"
-					(reference "#PWR054")
+					(reference "#PWR050")
 					(unit 1)
 				)
@@
 		(on_board yes)
 		(dnp no)
-		(property "Reference" "#PWR047"
+		(property "Reference" "#PWR045"
 			(at 64.77 113.03 0)
 			(effects
@@
 			(project "zynq7000"
 				(path "/b3b2a4a2-12d8-4419-9374-817f22e1ad00/b5d6f844-b9aa-4334-b3f0-dc08737c0a31"
-					(reference "#PWR047")
+					(reference "#PWR045")
 					(unit 1)
 				)
@@
 		(on_board yes)
 		(dnp no)
-		(property "Reference" "#PWR043"
+		(property "Reference" "#PWR042"
 			(at 105.41 50.8 0)
 			(effects
@@
 			(project "zynq7000"
 				(path "/b3b2a4a2-12d8-4419-9374-817f22e1ad00/b5d6f844-b9aa-4334-b3f0-dc08737c0a31"
-					(reference "#PWR043")
+					(reference "#PWR042")
 					(unit 1)
 				)
@@
 		(dnp no)
 		(fields_autoplaced yes)
-		(property "Reference" "#PWR046"
+		(property "Reference" "#PWR044"
 			(at 54.61 80.01 0)
 			(effects
@@
 			(project "zynq7000"
 				(path "/b3b2a4a2-12d8-4419-9374-817f22e1ad00/b5d6f844-b9aa-4334-b3f0-dc08737c0a31"
-					(reference "#PWR046")
+					(reference "#PWR044")
 					(unit 1)
 				)
@@
 		(on_board yes)
 		(dnp no)
-		(property "Reference" "R43"
+		(property "Reference" "R40"
 			(at 127 114.808 90)
 			(effects
@@
 			(project "zynq7000"
 				(path "/b3b2a4a2-12d8-4419-9374-817f22e1ad00/b5d6f844-b9aa-4334-b3f0-dc08737c0a31"
-					(reference "R43")
+					(reference "R40")
 					(unit 1)
 				)
@@
 		(on_board yes)
 		(dnp no)
-		(property "Reference" "R47"
+		(property "Reference" "R41"
 			(at 127 123.698 90)
 			(effects
@@
 			(project "zynq7000"
 				(path "/b3b2a4a2-12d8-4419-9374-817f22e1ad00/b5d6f844-b9aa-4334-b3f0-dc08737c0a31"
-					(reference "R47")
+					(reference "R41")
 					(unit 1)
 				)
@@
 		(dnp no)
 		(fields_autoplaced yes)
-		(property "Reference" "#PWR051"
+		(property "Reference" "#PWR048"
 			(at 48.26 129.54 0)
 			(effects
@@
 			(project "zynq7000"
 				(path "/b3b2a4a2-12d8-4419-9374-817f22e1ad00/b5d6f844-b9aa-4334-b3f0-dc08737c0a31"
-					(reference "#PWR051")
+					(reference "#PWR048")
 					(unit 1)
 				)
@@
 		(dnp no)
 		(fields_autoplaced yes)
-		(property "Reference" "#PWR057"
+		(property "Reference" "#PWR052"
 			(at 132.08 154.94 0)
 			(effects
@@
 			(project "zynq7000"
 				(path "/b3b2a4a2-12d8-4419-9374-817f22e1ad00/b5d6f844-b9aa-4334-b3f0-dc08737c0a31"
-					(reference "#PWR057")
+					(reference "#PWR052")
 					(unit 1)
 				)
@@
 		(on_board yes)
 		(dnp no)
-		(property "Reference" "R39"
+		(property "Reference" "R38"
 			(at 66.04 111.76 0)
 			(effects
@@
 			(project "zynq7000"
 				(path "/b3b2a4a2-12d8-4419-9374-817f22e1ad00/b5d6f844-b9aa-4334-b3f0-dc08737c0a31"
-					(reference "R39")
+					(reference "R38")
 					(unit 1)
 				)
@@
 		(on_board yes)
 		(dnp no)
-		(property "Reference" "#PWR044"
+		(property "Reference" "#PWR043"
 			(at 73.66 57.15 0)
 			(effects
@@
 			(project "zynq7000"
 				(path "/b3b2a4a2-12d8-4419-9374-817f22e1ad00/b5d6f844-b9aa-4334-b3f0-dc08737c0a31"
-					(reference "#PWR044")
+					(reference "#PWR043")
 					(unit 1)
 				)
@@
 		(dnp no)
 		(fields_autoplaced yes)
-		(property "Reference" "#PWR055"
+		(property "Reference" "#PWR051"
 			(at 45.72 147.32 0)
 			(effects
@@
 			(project "zynq7000"
 				(path "/b3b2a4a2-12d8-4419-9374-817f22e1ad00/b5d6f844-b9aa-4334-b3f0-dc08737c0a31"
-					(reference "#PWR055")
+					(reference "#PWR051")
 					(unit 1)
 				)

Commit message: update
Changed lines of the file:
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@@
 				)
 				(justify right)
+				(hide yes)
 			)
 		)
@@
 				)
 				(justify right)
+				(hide yes)
 			)
 		)
@@
 				)
 				(justify left)
+				(hide yes)
 			)
 		)
@@
 				)
 				(justify right)
+				(hide yes)
 			)
 		)
@@
 				)
 				(justify left)
+				(hide yes)
 			)
 		)
@@
 				)
 				(justify right)
+				(hide yes)
 			)
 		)
@@
 				)
 				(justify right)
+				(hide yes)
 			)
 		)
@@
 		(on_board yes)
 		(dnp no)
-		(fields_autoplaced yes)
 		(property "Reference" "SW2"
-			(at 52.07 125.73 0)
+			(at 44.45 128.27 0)
 			(effects
 				(font
@@
 		)
 		(property "Value" "SW_Push"
-			(at 52.07 128.27 0)
-			(effects
-				(font
+			(at 44.45 130.81 0)
+			(effects
+				(font
