File: pl_hdmi.kicad_sch (KiCad schematic)
At the start: 9 parts, among them J12 HDMI_A_1.4, Q1 2N7002, Q2 2N7002, Q3 2N7002

Commit message: add overview
Parts:
- renumbered R99 to R100, R95 to R96, R96 to R97, R97 to R98, R98 to R99
Changed lines of the file:
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@@
 				)
 				(justify right)
-				(hide yes)
 			)
 		)
@@
 				)
 				(justify right)
-				(hide yes)
 			)
 		)
@@
 				)
 				(justify right)
-				(hide yes)
 			)
 		)
@@
 				)
 				(justify right)
-				(hide yes)
 			)
 		)
@@
 				)
 				(justify right)
-				(hide yes)
 			)
 		)
@@
 				)
 				(justify right)
-				(hide yes)
 			)
 		)
@@
 				)
 				(justify right)
-				(hide yes)
 			)
 		)
@@
 				)
 				(justify right)
-				(hide yes)
 			)
 		)
@@
 				)
 				(justify right)
-				(hide yes)
 			)
 		)
@@
 				)
 				(justify right)
-				(hide yes)
 			)
 		)
@@
 				)
 				(justify right)
-				(hide yes)
 			)
 		)
@@
 				)
 				(justify right)
-				(hide yes)
 			)
 		)
@@
 		(on_board yes)
 		(dnp no)
-		(property "Reference" "R98"
+		(property "Reference" "R99"
 			(at 136.144 69.85 0)
 			(effects
@@
 			(project "zynq7000"
 				(path "/b3b2a4a2-12d8-4419-9374-817f22e1ad00/c765a720-2c44-4272-a581-62fbf9721656"
-					(reference "R98")
+					(reference "R99")
 					(unit 1)
 				)
@@
 		(dnp no)
 		(fields_autoplaced yes)
-		(property "Reference" "#PWR0214"
+		(property "Reference" "#PWR0229"
 			(at 91.44 125.73 0)
 			(effects
@@
 			(project "zynq7000"
 				(path "/b3b2a4a2-12d8-4419-9374-817f22e1ad00/c765a720-2c44-4272-a581-62fbf9721656"
-					(reference "#PWR0214")
+					(reference "#PWR0229")
 					(unit 1)
 				)
@@
 		(on_board yes)
 		(dnp no)
-		(property "Reference" "#PWR0211"
+		(property "Reference" "#PWR0226"
 			(at 137.16 67.31 0)
 			(effects
@@
 			(project "zynq7000"
 				(path "/b3b2a4a2-12d8-4419-9374-817f22e1ad00/c765a720-2c44-4272-a581-62fbf9721656"
-					(reference "#PWR0211")
+					(reference "#PWR0226")
 					(unit 1)
 				)
@@
 		(on_board yes)
 		(dnp no)
-		(property "Reference" "R95"
+		(property "Reference" "R96"
 			(at 86.106 69.85 0)
 			(effects
@@
 			(project "zynq7000"
 				(path "/b3b2a4a2-12d8-4419-9374-817f22e1ad00/c765a720-2c44-4272-a581-62fbf9721656"
-					(reference "R95")
+					(reference "R96")
 					(unit 1)
 				)
@@
 		(dnp no)
 		(fields_autoplaced yes)
-		(property "Reference" "#PWR0213"
+		(property "Reference" "#PWR0228"
 			(at 207.01 123.19 0)
 			(effects
@@
 			(project "zynq7000"
 				(path "/b3b2a4a2-12d8-4419-9374-817f22e1ad00/c765a720-2c44-4272-a581-62fbf9721656"
-					(reference "#PWR0213")
+					(reference "#PWR0228")
 					(unit 1)
 				)
@@
 		(on_board yes)
 		(dnp no)
-		(property "Reference" "R97"
+		(property "Reference" "R98"
 			(at 128.524 69.85 0)
 			(effects
@@
 			(project "zynq7000"
 				(path "/b3b2a4a2-12d8-4419-9374-817f22e1ad00/c765a720-2c44-4272-a581-62fbf9721656"
-					(reference "R97")
+					(reference "R98")
 					(unit 1)
 				)
@@
 		(on_board yes)
 		(dnp no)
-		(property "Reference" "#PWR0208"
+		(property "Reference" "#PWR0223"
 			(at 199.39 60.96 0)
 			(effects
@@
 			(project "zynq7000"
 				(path "/b3b2a4a2-12d8-4419-9374-817f22e1ad00/c765a720-2c44-4272-a581-62fbf9721656"
-					(reference "#PWR0208")
+					(reference "#PWR0223")
 					(unit 1)
 				)
@@
 		(on_board yes)
 		(dnp no)
-		(property "Reference" "#PWR0209"
+		(property "Reference" "#PWR0224"
 			(at 85.09 67.31 0)
 			(effects
@@
 			(project "zynq7000"
 				(path "/b3b2a4a2-12d8-4419-9374-817f22e1ad00/c765a720-2c44-4272-a581-62fbf9721656"
-					(reference "#PWR0209")
+					(reference "#PWR0224")
 					(unit 1)
 				)
@@
 		(on_board yes)
 		(dnp no)
-		(property "Reference" "#PWR0212"
+		(property "Reference" "#PWR0227"
 			(at 91.44 102.87 0)
 			(effects
@@
 			(project "zynq7000"
 				(path "/b3b2a4a2-12d8-4419-9374-817f22e1ad00/c765a720-2c44-4272-a581-62fbf9721656"
-					(reference "#PWR0212")
+					(reference "#PWR0227")
 					(unit 1)
 				)
@@
 		(on_board yes)
 		(dnp no)
-		(property "Reference" "#PWR0210"
+		(property "Reference" "#PWR0225"
 			(at 113.03 67.31 0)
 			(effects
@@
 			(project "zynq7000"
 				(path "/b3b2a4a2-12d8-4419-9374-817f22e1ad00/c765a720-2c44-4272-a581-62fbf9721656"
-					(reference "#PWR0210")
+					(reference "#PWR0225")
 					(unit 1)
 				)
@@
 		(on_board yes)
 		(dnp no)
-		(property "Reference" "R96"
+		(property "Reference" "R97"
 			(at 93.726 69.85 0)
 			(effects
@@
 			(project "zynq7000"
 				(path "/b3b2a4a2-12d8-4419-9374-817f22e1ad00/c765a720-2c44-4272-a581-62fbf9721656"
-					(reference "R96")
+					(reference "R97")
 					(unit 1)
 				)
@@
 		(on_board yes)
 		(dnp no)
-		(property "Reference" "R99"
+		(property "Reference" "R100"
 			(at 92.456 101.854 0)
 			(effects
@@
 			(project "zynq7000"
 				(path "/b3b2a4a2-12d8-4419-9374-817f22e1ad00/c765a720-2c44-4272-a581-62fbf9721656"
-					(reference "R99")
-					(unit 1)
-				)
+					(reference "R100")
+					(unit 1)
+				)
