File: pmic.kicad_sch (KiCad schematic)
At the start: 40 parts, among them IC1 MMPF0100NPAEP, J6 Header 2.54mm, SW3 SW_Push

Commit message: add overview
Parts:
- renumbered J6 to J5, R64 to R56, R65 to R57, R66 to R58, R67 to R59, R68 to R60

Commit message: update
Parts:
- added C174: 4u7, Capacitor_SMD:C_0402_1005Metric, symbol Device:C_Small
- added C175: 1u, Capacitor_SMD:C_0402_1005Metric, symbol Device:C_Small
- C59, C60, C61, C62, C63, C64, C65: value 4u7 -> 10u
- C79: value 1u -> 4u7
- C81: value 470n -> 1u
- C83: value 220n -> 1u
Connections:
- net +3V3: now also C175.1
- net GND: now also C174.2, C175.2
- net +1V8A: now reaches IC1.28 (VGEN4)
- net +1V8A: now also C174.1
- no-connect marks 11 -> 10
Other:
- note added: "populate when done programing"
- moved on the sheet: R59
