File: power_pins.kicad_sch (KiCad schematic)
At the start: 46 parts, among them U1 XC7Z010-1CLG400C

Commit message: update
Parts:
- added C173: 100u, Capacitor_SMD:C_1206_3216Metric, symbol Device:C_Small
- C100, C103, C106, C109, C112, C115, C119, C120, C121, C122, C124, C126, C127, C128, C129, C133, C134, C135, C136, C94, C95, C96, C99: value 470n -> 1u
Connections:
- net GND: now also C173.2
- net VCC_DDR: now also C173.1
Other:
- moved on the sheet: U1E
