File: ps_config.kicad_sch (KiCad schematic)
At the start: 11 parts, among them J4 Header 2.54mm, X1 ASE-40MHz

Commit message: add overview
Parts:
- renumbered C44 to C172, J4 to J13, R41 to R101, R42 to R102, R44 to R103, R45 to R104, R46 to R105, R49 to R106, R51 to R107, R36 to R108
Changed lines of the file:
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@@
 				)
 				(justify left)
-				(hide yes)
 			)
 		)
@@
 				)
 				(justify left)
-				(hide yes)
 			)
 		)
@@
 				)
 				(justify left)
-				(hide yes)
 			)
 		)
@@
 				)
 				(justify left)
-				(hide yes)
 			)
 		)
@@
 				)
 				(justify left)
-				(hide yes)
 			)
 		)
@@
 				)
 				(justify left)
-				(hide yes)
 			)
 		)
@@
 				)
 				(justify left)
-				(hide yes)
 			)
 		)
@@
 				)
 				(justify right)
-				(hide yes)
 			)
 		)
@@
 		(on_board yes)
 		(dnp no)
-		(property "Reference" "R41"
+		(property "Reference" "R101"
 			(at 206.5548 43.3624 90)
 			(effects
@@
 			(project "zynq7000"
 				(path "/b3b2a4a2-12d8-4419-9374-817f22e1ad00/17ba46b2-4fcf-4df1-9e0f-d12712bbed77"
-					(reference "R41")
+					(reference "R101")
 					(unit 1)
 				)
@@
 		(on_board yes)
 		(dnp no)
-		(property "Reference" "R49"
+		(property "Reference" "R106"
 			(at 191.3148 94.1624 90)
 			(effects
@@
 			(project "zynq7000"
 				(path "/b3b2a4a2-12d8-4419-9374-817f22e1ad00/17ba46b2-4fcf-4df1-9e0f-d12712bbed77"
-					(reference "R49")
+					(reference "R106")
 					(unit 1)
 				)
@@
 		(dnp no)
 		(fields_autoplaced yes)
-		(property "Reference" "J4"
+		(property "Reference" "J13"
 			(at 185.42 35.56 0)
 			(effects
@@
 			(project "zynq7000"
 				(path "/b3b2a4a2-12d8-4419-9374-817f22e1ad00/17ba46b2-4fcf-4df1-9e0f-d12712bbed77"
-					(reference "J4")
+					(reference "J13")
 					(unit 1)
 				)
@@
 		(on_board yes)
 		(dnp no)
-		(property "Reference" "#PWR056"
+		(property "Reference" "#PWR0232"
 			(at 184.15 97.79 0)
 			(effects
@@
 			(project "zynq7000"
 				(path "/b3b2a4a2-12d8-4419-9374-817f22e1ad00/17ba46b2-4fcf-4df1-9e0f-d12712bbed77"
-					(reference "#PWR056")
+					(reference "#PWR0232")
 					(unit 1)
 				)
@@
 		(on_board yes)
 		(dnp no)
-		(property "Reference" "R46"
+		(property "Reference" "R105"
 			(at 206.5548 53.5224 90)
 			(effects
@@
 			(project "zynq7000"
 				(path "/b3b2a4a2-12d8-4419-9374-817f22e1ad00/17ba46b2-4fcf-4df1-9e0f-d12712bbed77"
-					(reference "R46")
+					(reference "R105")
 					(unit 1)
 				)
@@
 		(on_board yes)
 		(dnp no)
-		(property "Reference" "R51"
+		(property "Reference" "R107"
 			(at 191.3148 96.7024 90)
 			(effects
@@
 			(project "zynq7000"
 				(path "/b3b2a4a2-12d8-4419-9374-817f22e1ad00/17ba46b2-4fcf-4df1-9e0f-d12712bbed77"
-					(reference "R51")
+					(reference "R107")
 					(unit 1)
 				)
@@
 		(dnp no)
 		(fields_autoplaced yes)
-		(property "Reference" "#PWR058"
+		(property "Reference" "#PWR0233"
 			(at 184.15 105.41 0)
 			(effects
@@
 			(project "zynq7000"
 				(path "/b3b2a4a2-12d8-4419-9374-817f22e1ad00/17ba46b2-4fcf-4df1-9e0f-d12712bbed77"
-					(reference "#PWR058")
+					(reference "#PWR0233")
 					(unit 1)
 				)
@@
 		(on_board yes)
 		(dnp no)
-		(property "Reference" "R45"
+		(property "Reference" "R104"
 			(at 206.5548 50.9824 90)
 			(effects
@@
 			(project "zynq7000"
 				(path "/b3b2a4a2-12d8-4419-9374-817f22e1ad00/17ba46b2-4fcf-4df1-9e0f-d12712bbed77"
-					(reference "R45")
+					(reference "R104")
 					(unit 1)
 				)
@@
 		(on_board yes)
 		(dnp no)
-		(property "Reference" "#PWR041"
+		(property "Reference" "#PWR0234"
 			(at 105.41 142.24 0)
 			(effects
@@
 			(project "zynq7000"
 				(path "/b3b2a4a2-12d8-4419-9374-817f22e1ad00/17ba46b2-4fcf-4df1-9e0f-d12712bbed77"
-					(reference "#PWR041")
+					(reference "#PWR0234")
 					(unit 1)
 				)
@@
 		(dnp no)
 		(fields_autoplaced yes)
-		(property "Reference" "#PWR045"
+		(property "Reference" "#PWR0235"
 			(at 105.41 162.56 0)
 			(effects
@@
 			(project "zynq7000"
 				(path "/b3b2a4a2-12d8-4419-9374-817f22e1ad00/17ba46b2-4fcf-4df1-9e0f-d12712bbed77"
-					(reference "#PWR045")
+					(reference "#PWR0235")
 					(unit 1)
 				)
@@
 		(dnp no)
 		(fields_autoplaced yes)
-		(property "Reference" "#PWR052"
+		(property "Reference" "#PWR0231"
 			(at 194.31 62.23 0)
 			(effects
@@
 			(project "zynq7000"
 				(path "/b3b2a4a2-12d8-4419-9374-817f22e1ad00/17ba46b2-4fcf-4df1-9e0f-d12712bbed77"
-					(reference "#PWR052")
+					(reference "#PWR0231")
 					(unit 1)
 				)
@@
 		(on_board yes)
 		(dnp no)
-		(property "Reference" "R36"
+		(property "Reference" "R108"
 			(at 92.71 149.352 90)
 			(effects
@@
 			(project "zynq7000"
 				(path "/b3b2a4a2-12d8-4419-9374-817f22e1ad00/17ba46b2-4fcf-4df1-9e0f-d12712bbed77"
-					(reference "R36")
+					(reference "R108")
 					(unit 1)
 				)
@@
 		(on_board yes)
 		(dnp no)
-		(property "Reference" "#PWR049"
+		(property "Reference" "#PWR0230"
 			(at 194.31 43.18 0)
 			(effects
@@
 			(project "zynq7000"
 				(path "/b3b2a4a2-12d8-4419-9374-817f22e1ad00/17ba46b2-4fcf-4df1-9e0f-d12712bbed77"
-					(reference "#PWR049")
+					(reference "#PWR0230")
 					(unit 1)
 				)
@@
 		(on_board yes)
 		(dnp no)
-		(property "Reference" "R42"
+		(property "Reference" "R102"
 			(at 206.5548 45.9024 90)
 			(effects
@@
 			(project "zynq7000"
 				(path "/b3b2a4a2-12d8-4419-9374-817f22e1ad00/17ba46b2-4fcf-4df1-9e0f-d12712bbed77"
-					(reference "R42")
+					(reference "R102")
 					(unit 1)
 				)
@@
 		(on_board yes)
 		(dnp no)
-		(property "Reference" "R44"
+		(property "Reference" "R103"
 			(at 206.5548 48.4424 90)
 			(effects
@@
 			(project "zynq7000"
 				(path "/b3b2a4a2-12d8-4419-9374-817f22e1ad00/17ba46b2-4fcf-4df1-9e0f-d12712bbed77"
-					(reference "R44")
+					(reference "R103")
 					(unit 1)
 				)
@@
 		(on_board yes)
 		(dnp no)
-		(property "Reference" "C44"
+		(property "Reference" "C172"
 			(at 117.348 149.86 0)
 			(effects
@@
 			(project "zynq7000"
 				(path "/b3b2a4a2-12d8-4419-9374-817f22e1ad00/17ba46b2-4fcf-4df1-9e0f-d12712bbed77"
-					(reference "C44")
-					(unit 1)
-				)
+					(reference "C172")
+					(unit 1)
+				)

Commit message: update
Parts:
- C172: value 470n -> 1u
- X1: value ASE-40MHz -> 40MHz
Changed lines of the file:
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@@
 				)
 				(justify left)
+				(hide yes)
 			)
 		)
@@
 				)
 				(justify left)
+				(hide yes)
 			)
 		)
@@
 				)
 				(justify left)
+				(hide yes)
 			)
 		)
@@
 				)
 				(justify left)
+				(hide yes)
 			)
 		)
@@
 				)
 				(justify left)
+				(hide yes)
 			)
 		)
@@
 				)
 				(justify left)
+				(hide yes)
 			)
 		)
@@
 				)
 				(justify left)
+				(hide yes)
 			)
 		)
@@
 				)
 				(justify right)
+				(hide yes)
 			)
 		)
@@
 			)
 		)
-		(property "Value" "ASE-40MHz"
+		(property "Value" "40MHz"
 			(at 97.282 140.208 0)
 			(effects
@@
 			)
 		)
-		(property "Value" "470n"
+		(property "Value" "1u"
 			(at 117.348 152.4 0)
 			(effects
