File: ps_dram_ct.kicad_sch (KiCad schematic)
At the start: 2 parts, among them J2 FPC 40 pins P0.5mm, U1 XC7Z010-1CLG400C

Commit message: add overview
Parts:
- removed J2: FPC 40 pins P0.5mm, Connector_FFC-FPC:Amphenol_F32Q-1A7x1-11040_1x40-1MP_P0.5mm_Horizontal, symbol Connector_Generic_MountingPin:Conn_01x40_MountingPin
- removed U1: XC7Z010-1CLG400C, Custom:CLG400_XIL-L, symbol Custom:XC7Z010-1CLG400C
- added C27, C28: 10n, Capacitor_SMD:C_0402_1005Metric, symbol Device:C_Small
- added R2, R5: 90R, Resistor_SMD:R_0402_1005Metric, symbol Device:R_Small
- added U1: XC7Z010-1CLG400C, Custom:CLG400_XIL-L, symbol Custom:XC7Z010-1CLG400C
Connections:
- net GND: now also C27.2, C28.2, R5.2
- new net: R2.2, U1.G5 (PS_DDR_VRN_502)
- new net: R5.1, U1.H5 (PS_DDR_VRP_502)
- new net DRAM_A0: U1.N2 (PS_DDR_A0_502)
- new net DRAM_A1: U1.K2 (PS_DDR_A1_502)
- new net DRAM_A10: U1.F5 (PS_DDR_A10_502)
- new net DRAM_A11: U1.G4 (PS_DDR_A11_502)
- new net DRAM_A12: U1.E4 (PS_DDR_A12_502)
- new net DRAM_A13: U1.D4 (PS_DDR_A13_502)
- new net DRAM_A14: U1.F4 (PS_DDR_A14_502)
- new net DRAM_A2: U1.M3 (PS_DDR_A2_502)
- new net DRAM_A3: U1.K3 (PS_DDR_A3_502)
- new net DRAM_A4: U1.M4 (PS_DDR_A4_502)
- new net DRAM_A5: U1.L1 (PS_DDR_A5_502)
- new net DRAM_A6: U1.L4 (PS_DDR_A6_502)
- new net DRAM_A7: U1.K4 (PS_DDR_A7_502)
- new net DRAM_A8: U1.K1 (PS_DDR_A8_502)
- new net DRAM_A9: U1.J4 (PS_DDR_A9_502)
- new net DRAM_BA0: U1.L5 (PS_DDR_BA0_502)
- new net DRAM_BA1: U1.R4 (PS_DDR_BA1_502)
- new net DRAM_BA2: U1.J5 (PS_DDR_BA2_502)
- new net DRAM_CASN: U1.P5 (PS_DDR_CAS_B_502)
- new net DRAM_CKE: U1.N3 (PS_DDR_CKE_502)
- new net DRAM_CLK_N: U1.M2 (PS_DDR_CKN_502)
- new net DRAM_CLK_P: U1.L2 (PS_DDR_CKP_502)
- new net DRAM_CSN: U1.N1 (PS_DDR_CS_B_502)
- new net DRAM_DM0: U1.A1 (PS_DDR_DM0_502)
- new net DRAM_DM1: U1.F1 (PS_DDR_DM1_502)
- new net DRAM_DQ0: U1.B3 (PS_DDR_DQ1_502)
- new net DRAM_DQ1: U1.D1 (PS_DDR_DQ5_502)
- new net DRAM_DQ10: U1.H2 (PS_DDR_DQ13_502)
- new net DRAM_DQ11: U1.J3 (PS_DDR_DQ12_502)
- new net DRAM_DQ12: U1.E2 (PS_DDR_DQ8_502)
- new net DRAM_DQ13: U1.J1 (PS_DDR_DQ15_502)
- new net DRAM_DQ14: U1.G3 (PS_DDR_DQ10_502)
- new net DRAM_DQ15: U1.H1 (PS_DDR_DQ14_502)
- new net DRAM_DQ2: U1.A4 (PS_DDR_DQ3_502)
- new net DRAM_DQ3: U1.D3 (PS_DDR_DQ4_502)
- new net DRAM_DQ4: U1.A2 (PS_DDR_DQ2_502)
- new net DRAM_DQ5: U1.E1 (PS_DDR_DQ7_502)
- new net DRAM_DQ6: U1.C3 (PS_DDR_DQ0_502)
- new net DRAM_DQ7: U1.C1 (PS_DDR_DQ6_502)
- new net DRAM_DQ8: U1.E3 (PS_DDR_DQ9_502)
- new net DRAM_DQ9: U1.H3 (PS_DDR_DQ11_502)
- new net DRAM_DQS0_N: U1.B2 (PS_DDR_DQS_N0_502)
- new net DRAM_DQS0_P: U1.C2 (PS_DDR_DQS_P0_502)
- new net DRAM_DQS1_N: U1.F2 (PS_DDR_DQS_N1_502)
- new net DRAM_DQS1_P: U1.G2 (PS_DDR_DQS_P1_502)
- new net DRAM_ODT: U1.N5 (PS_DDR_ODT_502)
- new net DRAM_RASN: U1.P4 (PS_DDR_RAS_B_502)
- new net DRAM_RSTN: U1.B4 (PS_DDR_DRST_B_502)
- new net DRAM_WEN: U1.M5 (PS_DDR_WE_B_502)
- new net VCC_DDR: R2.1
- new net VREF_DDR: C27.1, C28.1, U1.H6 (PS_DDR_VREF0_502), U1.P6 (PS_DDR_VREF1_502)
- no-connect marks 40 -> 22
Other:
- note added: "DRAM Controller"
- note removed: "Bank 35 IO pins (1.8V)"
- note removed: "Extended connector"

Commit message: update
Parts:
- C27, C28: value 10n -> 100n
- R2, R5: value 90R -> 120R
Other:
- moved on the sheet: R2, R5
