File: ps_eth.kicad_sch (KiCad schematic)
At the start: 34 parts, among them J9 HR911130A, U6 RTL8211F-CG, Y1 25MHz

Commit message: add overview
Parts:
- renumbered J9 to J8, R76 to R68, R77 to R69, R78 to R70, R79 to R71, R80 to R72, R81 to R73, R82 to R74, R83 to R75, R84 to R76, R85 to R77, R86 to R78, R87 to R79, R88 to R80, R89 to R81

Commit message: update
Parts:
- added R110: 10k, Resistor_SMD:R_0402_1005Metric, symbol Device:R_Small
- C143: value 470n -> 1u
- R78: value 2k49 -> 3k3
- U6: footprint Custom:RTL8211F-CG_RTK -> Custom:QFN_40_7x7mm_RTL8211F
Connections:
- net GND: now also R110.2
- net at R78.1, U6.39 (RSET): now also R110.1
Other:
- moved on the sheet: R78
Changed lines of the file:
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@@
 	)
 	(junction
+		(at 135.89 86.36)
+		(diameter 0)
+		(color 0 0 0 0)
+	)
+	(junction
 		(at 130.81 142.24)
 		(diameter 0)
@@
 	(wire
 		(pts
-			(xy 137.16 92.71) (xy 137.16 93.98)
+			(xy 135.89 92.71) (xy 135.89 93.98)
 		)
 		(stroke
@@
 	(wire
 		(pts
+			(xy 135.89 86.36) (xy 142.24 86.36)
+		)
+		(stroke
+			(width 0)
+			(type default)
+		)
+	)
+	(wire
+		(pts
 			(xy 80.01 144.78) (xy 80.01 142.24)
 		)
@@
 	(wire
 		(pts
-			(xy 137.16 86.36) (xy 135.89 86.36)
-		)
-		(stroke
-			(width 0)
-			(type default)
-		)
-	)
-	(wire
-		(pts
 			(xy 237.49 104.14) (xy 234.95 104.14)
 		)
@@
 	(wire
 		(pts
-			(xy 137.16 87.63) (xy 137.16 86.36)
+			(xy 135.89 87.63) (xy 135.89 86.36)
 		)
 		(stroke
@@
 	(wire
 		(pts
-			(xy 144.78 88.9) (xy 154.94 88.9)
+			(xy 146.05 88.9) (xy 154.94 88.9)
 		)
 		(stroke
@@
 	(wire
 		(pts
+			(xy 142.24 86.36) (xy 142.24 87.63)
+		)
+		(stroke
+			(width 0)
+			(type default)
+		)
+	)
+	(wire
+		(pts
 			(xy 234.95 33.02) (xy 241.3 33.02)
 		)
@@
 	(wire
 		(pts
-			(xy 144.78 96.52) (xy 154.94 96.52)
+			(xy 146.05 96.52) (xy 154.94 96.52)
 		)
 		(stroke
@@
 	(wire
 		(pts
+			(xy 142.24 92.71) (xy 142.24 93.98)
+		)
+		(stroke
+			(width 0)
+			(type default)
+		)
+	)
+	(wire
+		(pts
 			(xy 58.42 177.8) (xy 67.31 177.8)
 		)
@@
 	)
 	(label "ETH_LED0"
-		(at 144.78 88.9 0)
+		(at 146.05 88.9 0)
 		(effects
 			(font
@@
 	)
 	(label "ETH_LED2"
-		(at 144.78 96.52 0)
+		(at 146.05 96.52 0)
 		(effects
 			(font
@@
 				)
 				(justify right)
+				(hide yes)
 			)
 		)
@@
 				)
 				(justify right)
+				(hide yes)
 			)
 		)
@@
 				)
 				(justify right)
+				(hide yes)
 			)
 		)
@@
 				)
 				(justify right)
+				(hide yes)
 			)
 		)
@@
 				)
 				(justify right)
+				(hide yes)
 			)
 		)
@@
 				)
 				(justify right)
+				(hide yes)
 			)
 		)
@@
 				)
 				(justify right)
+				(hide yes)
 			)
 		)
@@
 				)
 				(justify right)
+				(hide yes)
 			)
 		)
@@
 				)
 				(justify right)
+				(hide yes)
 			)
 		)
@@
 				)
 				(justify right)
+				(hide yes)
 			)
 		)
@@
 				)
 				(justify right)
+				(hide yes)
 			)
 		)
@@
 				)
 				(justify right)
+				(hide yes)
 			)
 		)
@@
 				)
 				(justify right)
+				(hide yes)
 			)
 		)
@@
 				)
 				(justify right)
+				(hide yes)
 			)
 		)
@@
 	)
 	(symbol
+		(lib_id "Device:R_Small")
+		(at 142.24 90.17 0)
+		(unit 1)
+		(exclude_from_sim no)
+		(in_bom yes)
+		(on_board yes)
+		(dnp no)
+		(property "Reference" "R110"
+			(at 143.51 90.17 0)
+			(effects
+				(font
+					(size 1.016 1.016)
+				)
+				(justify left)
+			)
+		)
+		(property "Value" "10k"
+			(at 143.51 92.7099 0)
+			(effects
+				(font
+					(size 1.27 1.27)
+				)
+				(justify left)
+			)
+		)
+		(property "Footprint" "Resistor_SMD:R_0402_1005Metric"
+			(at 142.24 90.17 0)
+			(effects
+				(font
+					(size 1.27 1.27)
+				)
+				(hide yes)
+			)
+		)
+		(property "Datasheet" "~"
+			(at 142.24 90.17 0)
+			(effects
+				(font
+					(size 1.27 1.27)
+				)
+				(hide yes)
+			)
+		)
+		(property "Description" "Resistor, small symbol"
+			(at 142.24 90.17 0)
+			(effects
+				(font
+					(size 1.27 1.27)
+				)
+				(hide yes)
+			)
+		)
+		(pin "2"
+		)
+		(pin "1"
+		)
+		(instances
+			(project "zynq7000"
+				(path "/b3b2a4a2-12d8-4419-9374-817f22e1ad00/31d07f50-4c9a-4d57-85cb-b827351d4860"
+					(reference "R110")
+					(unit 1)
+				)
+			)
+		)
+	)
+	(symbol
 		(lib_id "Device:C_Small")
 		(at 123.19 146.05 0)
@@
 			)
 		)
-		(property "Value" "470n"
+		(property "Value" "1u"
 			(at 125.73 147.3262 0)
 			(effects
@@
 			)
 		)
-		(property "Footprint" "Custom:RTL8211F-CG_RTK"
+		(property "Footprint" "Custom:QFN_40_7x7mm_RTL8211F"
 			(at 93.98 35.56 0)
 			(effects
@@
 	(symbol
 		(lib_id "power:GND")
+		(at 142.24 93.98 0)
+		(unit 1)
+		(exclude_from_sim no)
+		(in_bom yes)
+		(on_board yes)
+		(dnp no)
+		(fields_autoplaced yes)
+		(property "Reference" "#PWR0242"
+			(at 142.24 100.33 0)
+			(effects
+				(font
+					(size 1.27 1.27)
+				)
+				(hide yes)
+			)
+		)
+		(property "Value" "GND"
+			(at 142.24 99.06 0)
+			(effects
+				(font
+					(size 1.27 1.27)
+				)
+				(hide yes)
+			)
+		)
+		(property "Footprint" ""
+			(at 142.24 93.98 0)
+			(effects
+				(font
+					(size 1.27 1.27)
+				)
+				(hide yes)
+			)
+		)
+		(property "Datasheet" ""
+			(at 142.24 93.98 0)
+			(effects
+				(font
+					(size 1.27 1.27)
+				)
+				(hide yes)
+			)
+		)
+		(property "Description" "Power symbol creates a global label with name \"GND\" , ground"
+			(at 142.24 93.98 0)
+			(effects
+				(font
+					(size 1.27 1.27)
+				)
+				(hide yes)
+			)
+		)
+		(pin "1"
+		)
+		(instances
+			(project "zynq7000"
+				(path "/b3b2a4a2-12d8-4419-9374-817f22e1ad00/31d07f50-4c9a-4d57-85cb-b827351d4860"
+					(reference "#PWR0242")
+					(unit 1)
+				)
+			)
+		)
+	)
+	(symbol
+		(lib_id "power:GND")
 		(at 241.3 71.12 0)
 		(unit 1)
@@
 			)
 		)
-		(property "Footprint" "Custom:RTL8211F-CG_RTK"
+		(property "Footprint" "Custom:QFN_40_7x7mm_RTL8211F"
 			(at 85.09 139.7 0)
 			(effects
@@
 	(symbol
 		(lib_id "Device:R_Small")
-		(at 137.16 90.17 0)
+		(at 135.89 90.17 0)
 		(unit 1)
 		(exclude_from_sim no)
@@
 		(dnp no)
 		(property "Reference" "R78"
-			(at 138.43 88.9 0)
+			(at 137.16 88.9 0)
 			(effects
 				(font
@@
 			)
 		)
-		(property "Value" "2k49"
-			(at 138.43 91.4399 0)
+		(property "Value" "3k3"
+			(at 137.16 91.4399 0)
 			(effects
 				(font
@@
 		)
 		(property "Footprint" "Resistor_SMD:R_0402_1005Metric"
-			(at 137.16 90.17 0)
+			(at 135.89 90.17 0)
 			(effects
 				(font
@@
 		)
 		(property "Datasheet" "~"
-			(at 137.16 90.17 0)
+			(at 135.89 90.17 0)
 			(effects
 				(font
@@
 		)
 		(property "Description" "Resistor, small symbol"
-			(at 137.16 90.17 0)
+			(at 135.89 90.17 0)
 			(effects
 				(font
@@
 	(symbol
 		(lib_id "power:GND")
-		(at 137.16 93.98 0)
+		(at 135.89 93.98 0)
 		(unit 1)
 		(exclude_from_sim no)
@@
 		(fields_autoplaced yes)
 		(property "Reference" "#PWR0170"
-			(at 137.16 100.33 0)
+			(at 135.89 100.33 0)
 			(effects
 				(font
@@
 		)
 		(property "Value" "GND"
-			(at 137.16 99.06 0)
+			(at 135.89 99.06 0)
 			(effects
 				(font
@@
 		)
 		(property "Footprint" ""
-			(at 137.16 93.98 0)
+			(at 135.89 93.98 0)
 			(effects
 				(font
@@
 		)
 		(property "Datasheet" ""
-			(at 137.16 93.98 0)
+			(at 135.89 93.98 0)
 			(effects
 				(font
@@
 		)
 		(property "Description" "Power symbol creates a global label with name \"GND\" , ground"
-			(at 137.16 93.98 0)
+			(at 135.89 93.98 0)
 			(effects
 				(font
@@
 					(size 1.27 1.27)
 				)
+				(hide yes)
 			)
 		)
