File: ps_gpio.kicad_sch (KiCad schematic)
At the start: 12 parts, among them U1 XC7Z010-1CLG400C

Commit message: add overview
Parts:
- renumbered R52 to R44, R53 to R45, R54 to R46, R55 to R47, R56 to R48, R57 to R49, R58 to R50, R59 to R51, R60 to R52
Changed lines of the file:
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@@
 				)
 				(justify right)
-				(hide yes)
 			)
 		)
@@
 				)
 				(justify right)
-				(hide yes)
 			)
 		)
@@
 				)
 				(justify left)
-				(hide yes)
 			)
 		)
@@
 				)
 				(justify left)
-				(hide yes)
 			)
 		)
@@
 				)
 				(justify left)
-				(hide yes)
 			)
 		)
@@
 				)
 				(justify right)
-				(hide yes)
 			)
 		)
@@
 				)
 				(justify left)
-				(hide yes)
 			)
 		)
@@
 				)
 				(justify right)
-				(hide yes)
 			)
 		)
@@
 				)
 				(justify right)
-				(hide yes)
 			)
 		)
@@
 				)
 				(justify right)
-				(hide yes)
 			)
 		)
@@
 				)
 				(justify left)
-				(hide yes)
 			)
 		)
@@
 				)
 				(justify right)
-				(hide yes)
 			)
 		)
@@
 				)
 				(justify left)
-				(hide yes)
 			)
 		)
@@
 				)
 				(justify left)
-				(hide yes)
 			)
 		)
@@
 				)
 				(justify left)
-				(hide yes)
 			)
 		)
@@
 				)
 				(justify left)
-				(hide yes)
 			)
 		)
@@
 				)
 				(justify left)
-				(hide yes)
 			)
 		)
@@
 				)
 				(justify left)
-				(hide yes)
 			)
 		)
@@
 				)
 				(justify left)
-				(hide yes)
 			)
 		)
@@
 				)
 				(justify right)
-				(hide yes)
 			)
 		)
@@
 				)
 				(justify left)
-				(hide yes)
 			)
 		)
@@
 				)
 				(justify left)
-				(hide yes)
 			)
 		)
@@
 				)
 				(justify left)
-				(hide yes)
 			)
 		)
@@
 				)
 				(justify left)
-				(hide yes)
 			)
 		)
@@
 				)
 				(justify right)
-				(hide yes)
 			)
 		)
@@
 				)
 				(justify right)
-				(hide yes)
 			)
 		)
@@
 				)
 				(justify left)
-				(hide yes)
 			)
 		)
@@
 				)
 				(justify left)
-				(hide yes)
 			)
 		)
@@
 				)
 				(justify right)
-				(hide yes)
 			)
 		)
@@
 				)
 				(justify left)
-				(hide yes)
 			)
 		)
@@
 				)
 				(justify left)
-				(hide yes)
 			)
 		)
@@
 				)
 				(justify left)
-				(hide yes)
 			)
 		)
@@
 				)
 				(justify right)
-				(hide yes)
 			)
 		)
@@
 				)
 				(justify left)
-				(hide yes)
 			)
 		)
@@
 				)
 				(justify right)
-				(hide yes)
 			)
 		)
@@
 				)
 				(justify right)
-				(hide yes)
 			)
 		)
@@
 				)
 				(justify left)
-				(hide yes)
 			)
 		)
@@
 				)
 				(justify right)
-				(hide yes)
 			)
 		)
@@
 				)
 				(justify left)
-				(hide yes)
 			)
 		)
@@
 				)
 				(justify right)
-				(hide yes)
 			)
 		)
@@
 				)
 				(justify left)
-				(hide yes)
 			)
 		)
@@
 				)
 				(justify left)
-				(hide yes)
 			)
 		)
@@
 		(dnp no)
 		(fields_autoplaced yes)
-		(property "Reference" "#PWR060"
+		(property "Reference" "#PWR054"
 			(at 69.85 95.25 0)
 			(effects
@@
 			(project ""
 				(path "/b3b2a4a2-12d8-4419-9374-817f22e1ad00/6e41b7a2-4b5b-470c-a751-97a4cb58da79"
-					(reference "#PWR060")
+					(reference "#PWR054")
 					(unit 1)
 				)
@@
 		(on_board yes)
 		(dnp no)
-		(property "Reference" "R52"
+		(property "Reference" "R44"
 			(at 193.04 38.1 90)
 			(effects
@@
 			(project "zynq7000"
 				(path "/b3b2a4a2-12d8-4419-9374-817f22e1ad00/6e41b7a2-4b5b-470c-a751-97a4cb58da79"
-					(reference "R52")
+					(reference "R44")
 					(unit 1)
 				)
@@
 		(on_board yes)
 		(dnp no)
-		(property "Reference" "R54"
+		(property "Reference" "R46"
 			(at 193.04 43.18 90)
 			(effects
@@
 			(project "zynq7000"
 				(path "/b3b2a4a2-12d8-4419-9374-817f22e1ad00/6e41b7a2-4b5b-470c-a751-97a4cb58da79"
-					(reference "R54")
+					(reference "R46")
 					(unit 1)
 				)
@@
 		(dnp no)
 		(fields_autoplaced yes)
-		(property "Reference" "R60"
+		(property "Reference" "R52"
 			(at 83.82 96.52 90)
 			(effects
@@
 			(project ""
 				(path "/b3b2a4a2-12d8-4419-9374-817f22e1ad00/6e41b7a2-4b5b-470c-a751-97a4cb58da79"
-					(reference "R60")
+					(reference "R52")
 					(unit 1)
 				)
@@
 		(dnp no)
 		(fields_autoplaced yes)
-		(property "Reference" "#PWR061"
+		(property "Reference" "#PWR055"
 			(at 95.25 109.22 0)
 			(effects
@@
 			(project ""
 				(path "/b3b2a4a2-12d8-4419-9374-817f22e1ad00/6e41b7a2-4b5b-470c-a751-97a4cb58da79"
-					(reference "#PWR061")
+					(reference "#PWR055")
 					(unit 1)
 				)
@@
 		(on_board yes)
 		(dnp no)
-		(property "Reference" "R55"
+		(property "Reference" "R47"
 			(at 193.04 45.72 90)
 			(effects
@@
 			(project "zynq7000"
 				(path "/b3b2a4a2-12d8-4419-9374-817f22e1ad00/6e41b7a2-4b5b-470c-a751-97a4cb58da79"
-					(reference "R55")
+					(reference "R47")
 					(unit 1)
 				)
@@
 		(on_board yes)
 		(dnp no)
-		(property "Reference" "R58"
+		(property "Reference" "R50"
 			(at 71.12 74.93 0)
 			(effects
@@
 			(project ""
 				(path "/b3b2a4a2-12d8-4419-9374-817f22e1ad00/6e41b7a2-4b5b-470c-a751-97a4cb58da79"
-					(reference "R58")
+					(reference "R50")
 					(unit 1)
 				)
@@
 		(on_board yes)
 		(dnp no)
-		(property "Reference" "R57"
+		(property "Reference" "R49"
 			(at 193.04 50.8 90)
 			(effects
@@
 			(project "zynq7000"
 				(path "/b3b2a4a2-12d8-4419-9374-817f22e1ad00/6e41b7a2-4b5b-470c-a751-97a4cb58da79"
-					(reference "R57")
+					(reference "R49")
 					(unit 1)
 				)
@@
 		(on_board yes)
 		(dnp no)
-		(property "Reference" "R59"
+		(property "Reference" "R51"
 			(at 71.12 82.55 0)
 			(effects
@@
 			(project "zynq7000"
 				(path "/b3b2a4a2-12d8-4419-9374-817f22e1ad00/6e41b7a2-4b5b-470c-a751-97a4cb58da79"
-					(reference "R59")
+					(reference "R51")
 					(unit 1)
 				)
@@
 		(on_board yes)
 		(dnp no)
-		(property "Reference" "#PWR059"
+		(property "Reference" "#PWR053"
 			(at 69.85 76.2 0)
 			(effects
@@
 			(project ""
 				(path "/b3b2a4a2-12d8-4419-9374-817f22e1ad00/6e41b7a2-4b5b-470c-a751-97a4cb58da79"
-					(reference "#PWR059")
+					(reference "#PWR053")
 					(unit 1)
 				)
@@
 		(on_board yes)
 		(dnp no)
-		(property "Reference" "R56"
+		(property "Reference" "R48"
 			(at 193.04 48.26 90)
 			(effects
@@
 			(project "zynq7000"
 				(path "/b3b2a4a2-12d8-4419-9374-817f22e1ad00/6e41b7a2-4b5b-470c-a751-97a4cb58da79"
-					(reference "R56")
+					(reference "R48")
 					(unit 1)
 				)
@@
 		(on_board yes)
 		(dnp no)
-		(property "Reference" "R53"
+		(property "Reference" "R45"
 			(at 193.04 40.64 90)
 			(effects
@@
 			(project "zynq7000"
 				(path "/b3b2a4a2-12d8-4419-9374-817f22e1ad00/6e41b7a2-4b5b-470c-a751-97a4cb58da79"
-					(reference "R53")
+					(reference "R45")
 					(unit 1)
 				)

Commit message: update
Parts:
- C47: value 10n -> 100n
Connections:
- net SDIO1_CLK: now also U1.D9 (PS_MIO12_500); no longer U1.E9 (PS_MIO10_500)
- net SDIO1_D0: now also U1.E9 (PS_MIO10_500); no longer U1.D9 (PS_MIO12_500)
