File: ps_sd_qspi.kicad_sch (KiCad schematic)
At the start: 4 parts, among them J11 Micro_SD_Card_Det1, U8 W25Q128JVS

Commit message: add overview
Parts:
- renumbered J11 to J10, R94 to R86
Changed lines of the file:
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@@
 				)
 				(justify right)
-				(hide yes)
 			)
 		)
@@
 				)
 				(justify right)
-				(hide yes)
 			)
 		)
@@
 				)
 				(justify right)
-				(hide yes)
 			)
 		)
@@
 				)
 				(justify right)
-				(hide yes)
 			)
 		)
@@
 				)
 				(justify right)
-				(hide yes)
 			)
 		)
@@
 				)
 				(justify right)
-				(hide yes)
 			)
 		)
@@
 				)
 				(justify right)
-				(hide yes)
 			)
 		)
@@
 				)
 				(justify right)
-				(hide yes)
 			)
 		)
@@
 				)
 				(justify right)
-				(hide yes)
 			)
 		)
@@
 				)
 				(justify right)
-				(hide yes)
 			)
 		)
@@
 				)
 				(justify right)
-				(hide yes)
 			)
 		)
@@
 				)
 				(justify right)
-				(hide yes)
 			)
 		)
@@
 				)
 				(justify right)
-				(hide yes)
 			)
 		)
@@
 		(dnp no)
 		(fields_autoplaced yes)
-		(property "Reference" "#PWR0203"
+		(property "Reference" "#PWR0197"
 			(at 209.55 85.09 0)
 			(effects
@@
 			(project "zynq7000"
 				(path "/b3b2a4a2-12d8-4419-9374-817f22e1ad00/155597a2-50fa-4c69-90e9-c67747b47d74"
-					(reference "#PWR0203")
+					(reference "#PWR0197")
 					(unit 1)
 				)
@@
 		(dnp no)
 		(fields_autoplaced yes)
-		(property "Reference" "#PWR0206"
+		(property "Reference" "#PWR0200"
 			(at 193.04 104.14 0)
 			(effects
@@
 			(project "zynq7000"
 				(path "/b3b2a4a2-12d8-4419-9374-817f22e1ad00/155597a2-50fa-4c69-90e9-c67747b47d74"
-					(reference "#PWR0206")
+					(reference "#PWR0200")
 					(unit 1)
 				)
@@
 		(on_board yes)
 		(dnp no)
-		(property "Reference" "#PWR0202"
+		(property "Reference" "#PWR0196"
 			(at 193.04 72.39 0)
 			(effects
@@
 			(project "zynq7000"
 				(path "/b3b2a4a2-12d8-4419-9374-817f22e1ad00/155597a2-50fa-4c69-90e9-c67747b47d74"
-					(reference "#PWR0202")
+					(reference "#PWR0196")
 					(unit 1)
 				)
@@
 		(on_board yes)
 		(dnp no)
-		(property "Reference" "#PWR0204"
+		(property "Reference" "#PWR0198"
 			(at 78.74 81.28 0)
 			(effects
@@
 			(project "zynq7000"
 				(path "/b3b2a4a2-12d8-4419-9374-817f22e1ad00/155597a2-50fa-4c69-90e9-c67747b47d74"
-					(reference "#PWR0204")
+					(reference "#PWR0198")
 					(unit 1)
 				)
@@
 		(dnp no)
 		(fields_autoplaced yes)
-		(property "Reference" "J11"
+		(property "Reference" "J10"
 			(at 99.695 62.23 0)
 			(effects
@@
 			(project "zynq7000"
 				(path "/b3b2a4a2-12d8-4419-9374-817f22e1ad00/155597a2-50fa-4c69-90e9-c67747b47d74"
-					(reference "J11")
+					(reference "J10")
 					(unit 1)
 				)
@@
 		(dnp no)
 		(fields_autoplaced yes)
-		(property "Reference" "#PWR0205"
+		(property "Reference" "#PWR0199"
 			(at 74.93 104.14 0)
 			(effects
@@
 			(project "zynq7000"
 				(path "/b3b2a4a2-12d8-4419-9374-817f22e1ad00/155597a2-50fa-4c69-90e9-c67747b47d74"
-					(reference "#PWR0205")
+					(reference "#PWR0199")
 					(unit 1)
 				)
@@
 		(on_board yes)
 		(dnp no)
-		(property "Reference" "#PWR0207"
+		(property "Reference" "#PWR0201"
 			(at 62.23 110.49 0)
 			(effects
@@
 			(project "zynq7000"
 				(path "/b3b2a4a2-12d8-4419-9374-817f22e1ad00/155597a2-50fa-4c69-90e9-c67747b47d74"
-					(reference "#PWR0207")
+					(reference "#PWR0201")
 					(unit 1)
 				)
@@
 		(on_board yes)
 		(dnp no)
-		(property "Reference" "R94"
+		(property "Reference" "R86"
 			(at 69.85 101.6 0)
 			(effects
@@
 			(project "zynq7000"
 				(path "/b3b2a4a2-12d8-4419-9374-817f22e1ad00/155597a2-50fa-4c69-90e9-c67747b47d74"
-					(reference "R94")
+					(reference "R86")
 					(unit 1)
 				)
