File: ps_usb.kicad_sch (KiCad schematic)
At the start: 11 parts, among them J10 USB_C_Receptacle_USB2.0_16P, U7 USB3320C-EZK-TR

Commit message: add overview
Parts:
- renumbered J10 to J9, R90 to R82, R91 to R83, R92 to R84, R93 to R85
Changed lines of the file:
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@@
 				)
 				(justify right)
-				(hide yes)
 			)
 		)
@@
 				)
 				(justify right)
-				(hide yes)
 			)
 		)
@@
 				)
 				(justify right)
-				(hide yes)
 			)
 		)
@@
 				)
 				(justify right)
-				(hide yes)
 			)
 		)
@@
 				)
 				(justify right)
-				(hide yes)
 			)
 		)
@@
 				)
 				(justify right)
-				(hide yes)
 			)
 		)
@@
 				)
 				(justify right)
-				(hide yes)
 			)
 		)
@@
 				)
 				(justify right)
-				(hide yes)
 			)
 		)
@@
 				)
 				(justify right)
-				(hide yes)
 			)
 		)
@@
 				)
 				(justify right)
-				(hide yes)
 			)
 		)
@@
 				)
 				(justify right)
-				(hide yes)
 			)
 		)
@@
 				)
 				(justify right)
-				(hide yes)
 			)
 		)
@@
 		(dnp no)
 		(fields_autoplaced yes)
-		(property "Reference" "#PWR0194"
+		(property "Reference" "#PWR0188"
 			(at 142.24 80.01 0)
 			(effects
@@
 			(project "zynq7000"
 				(path "/b3b2a4a2-12d8-4419-9374-817f22e1ad00/425f6627-498e-46fb-bca9-bc293c9f13f9"
-					(reference "#PWR0194")
+					(reference "#PWR0188")
 					(unit 1)
 				)
@@
 		(dnp no)
 		(fields_autoplaced yes)
-		(property "Reference" "#PWR0197"
+		(property "Reference" "#PWR0191"
 			(at 166.37 90.17 0)
 			(effects
@@
 			(project "zynq7000"
 				(path "/b3b2a4a2-12d8-4419-9374-817f22e1ad00/425f6627-498e-46fb-bca9-bc293c9f13f9"
-					(reference "#PWR0197")
+					(reference "#PWR0191")
 					(unit 1)
 				)
@@
 		(on_board yes)
 		(dnp no)
-		(property "Reference" "#PWR0195"
+		(property "Reference" "#PWR0189"
 			(at 177.8 77.47 0)
 			(effects
@@
 			(project "zynq7000"
 				(path "/b3b2a4a2-12d8-4419-9374-817f22e1ad00/425f6627-498e-46fb-bca9-bc293c9f13f9"
-					(reference "#PWR0195")
+					(reference "#PWR0189")
 					(unit 1)
 				)
@@
 		(on_board yes)
 		(dnp no)
-		(property "Reference" "#PWR0198"
+		(property "Reference" "#PWR0192"
 			(at 152.4 92.71 0)
 			(effects
@@
 			(project "zynq7000"
 				(path "/b3b2a4a2-12d8-4419-9374-817f22e1ad00/425f6627-498e-46fb-bca9-bc293c9f13f9"
-					(reference "#PWR0198")
+					(reference "#PWR0192")
 					(unit 1)
 				)
@@
 		(dnp no)
 		(fields_autoplaced yes)
-		(property "Reference" "#PWR0193"
+		(property "Reference" "#PWR0187"
 			(at 113.03 80.01 0)
 			(effects
@@
 			(project "zynq7000"
 				(path "/b3b2a4a2-12d8-4419-9374-817f22e1ad00/425f6627-498e-46fb-bca9-bc293c9f13f9"
-					(reference "#PWR0193")
+					(reference "#PWR0187")
 					(unit 1)
 				)
@@
 		(on_board yes)
 		(dnp no)
-		(property "Reference" "R92"
+		(property "Reference" "R84"
 			(at 173.99 78.74 90)
 			(effects
@@
 			(project "zynq7000"
 				(path "/b3b2a4a2-12d8-4419-9374-817f22e1ad00/425f6627-498e-46fb-bca9-bc293c9f13f9"
-					(reference "R92")
+					(reference "R84")
 					(unit 1)
 				)
@@
 		(on_board yes)
 		(dnp no)
-		(property "Reference" "J10"
+		(property "Reference" "J9"
 			(at 186.69 68.58 0)
 			(effects
@@
 			(project "zynq7000"
 				(path "/b3b2a4a2-12d8-4419-9374-817f22e1ad00/425f6627-498e-46fb-bca9-bc293c9f13f9"
-					(reference "J10")
+					(reference "J9")
 					(unit 1)
 				)
@@
 		(on_board yes)
 		(dnp no)
-		(property "Reference" "R91"
+		(property "Reference" "R83"
 			(at 173.99 76.2 90)
 			(effects
@@
 			(project "zynq7000"
 				(path "/b3b2a4a2-12d8-4419-9374-817f22e1ad00/425f6627-498e-46fb-bca9-bc293c9f13f9"
-					(reference "R91")
+					(reference "R83")
 					(unit 1)
 				)
@@
 		(on_board yes)
 		(dnp no)
-		(property "Reference" "#PWR0191"
+		(property "Reference" "#PWR0185"
 			(at 149.86 68.58 0)
 			(effects
@@
 			(project "zynq7000"
 				(path "/b3b2a4a2-12d8-4419-9374-817f22e1ad00/425f6627-498e-46fb-bca9-bc293c9f13f9"
-					(reference "#PWR0191")
+					(reference "#PWR0185")
 					(unit 1)
 				)
@@
 		(on_board yes)
 		(dnp no)
-		(property "Reference" "#PWR0190"
+		(property "Reference" "#PWR0184"
 			(at 142.24 68.58 0)
 			(effects
@@
 			(project "zynq7000"
 				(path "/b3b2a4a2-12d8-4419-9374-817f22e1ad00/425f6627-498e-46fb-bca9-bc293c9f13f9"
-					(reference "#PWR0190")
+					(reference "#PWR0184")
 					(unit 1)
 				)
@@
 		(dnp no)
 		(fields_autoplaced yes)
-		(property "Reference" "#PWR0199"
+		(property "Reference" "#PWR0193"
 			(at 156.21 123.19 0)
 			(effects
@@
 			(project "zynq7000"
 				(path "/b3b2a4a2-12d8-4419-9374-817f22e1ad00/425f6627-498e-46fb-bca9-bc293c9f13f9"
-					(reference "#PWR0199")
+					(reference "#PWR0193")
 					(unit 1)
 				)
@@
 		(dnp no)
 		(fields_autoplaced yes)
-		(property "Reference" "#PWR0200"
+		(property "Reference" "#PWR0194"
 			(at 203.2 123.19 0)
 			(effects
@@
 			(project "zynq7000"
 				(path "/b3b2a4a2-12d8-4419-9374-817f22e1ad00/425f6627-498e-46fb-bca9-bc293c9f13f9"
-					(reference "#PWR0200")
+					(reference "#PWR0194")
 					(unit 1)
 				)
@@
 		(on_board yes)
 		(dnp no)
-		(property "Reference" "#PWR0192"
+		(property "Reference" "#PWR0186"
 			(at 124.46 76.2 0)
 			(effects
@@
 			(project "zynq7000"
 				(path "/b3b2a4a2-12d8-4419-9374-817f22e1ad00/425f6627-498e-46fb-bca9-bc293c9f13f9"
-					(reference "#PWR0192")
+					(reference "#PWR0186")
 					(unit 1)
 				)
@@
 		(dnp no)
 		(fields_autoplaced yes)
-		(property "Reference" "#PWR0196"
+		(property "Reference" "#PWR0190"
 			(at 149.86 81.28 0)
 			(effects
@@
 			(project "zynq7000"
 				(path "/b3b2a4a2-12d8-4419-9374-817f22e1ad00/425f6627-498e-46fb-bca9-bc293c9f13f9"
-					(reference "#PWR0196")
+					(reference "#PWR0190")
 					(unit 1)
 				)
@@
 		(on_board yes)
 		(dnp no)
-		(property "Reference" "#PWR0189"
+		(property "Reference" "#PWR0183"
 			(at 113.03 67.31 0)
 			(effects
@@
 			(project "zynq7000"
 				(path "/b3b2a4a2-12d8-4419-9374-817f22e1ad00/425f6627-498e-46fb-bca9-bc293c9f13f9"
-					(reference "#PWR0189")
+					(reference "#PWR0183")
 					(unit 1)
 				)
@@
 		(on_board yes)
 		(dnp no)
-		(property "Reference" "R93"
+		(property "Reference" "R85"
 			(at 157.48 109.22 0)
 			(effects
@@
 			(project "zynq7000"
 				(path "/b3b2a4a2-12d8-4419-9374-817f22e1ad00/425f6627-498e-46fb-bca9-bc293c9f13f9"
-					(reference "R93")
+					(reference "R85")
 					(unit 1)
 				)
@@
 		(on_board yes)
 		(dnp no)
-		(property "Reference" "#PWR0201"
+		(property "Reference" "#PWR0195"
 			(at 97.79 125.73 0)
 			(effects
@@
 			(project "zynq7000"
 				(path "/b3b2a4a2-12d8-4419-9374-817f22e1ad00/425f6627-498e-46fb-bca9-bc293c9f13f9"
-					(reference "#PWR0201")
+					(reference "#PWR0195")
 					(unit 1)
 				)
@@
 		(on_board yes)
 		(dnp no)
-		(property "Reference" "R90"
+		(property "Reference" "R82"
 			(at 135.89 68.58 0)
 			(effects
@@
 			(project "zynq7000"
 				(path "/b3b2a4a2-12d8-4419-9374-817f22e1ad00/425f6627-498e-46fb-bca9-bc293c9f13f9"
-					(reference "R90")
-					(unit 1)
-				)
+					(reference "R82")
+					(unit 1)
+				)

Commit message: update
Parts:
- added R109: 1k2, Resistor_SMD:R_0402_1005Metric, symbol Device:R_Small
- C151: value 2u2 -> 4u7
- R85: value 8k06 -> 6k8
- U7: footprint Custom:QFN32_5X5MC_MCH -> Custom:QFN32_5X5_USB3320
Connections:
- net GND: now also R109.2; no longer R85.2
- new net: R109.1, R85.2
