File: zynq7000.kicad_sch (KiCad schematic)
At the start: 4 parts

Commit message: add overview
Other:
- added sheet DRAM Controller (ps_dram_ct.kicad_sch)
- note added: "Audio CODEC"
- note added: "Audio Jack"
- note added: "Bank 34 IO (3.3V)"
- note added: "Bank 35 IO (1.8V)"
- note added: "Battery 2000mAh"
- note added: "Battery Charger"
- note added: "DRAM Controller"
- note added: "DRAM DDR3"
- note added: "FPC Connector"
- note added: "FTDI USB - JTAG"
- note added: "Gigabit Ethernet PHY"
- note added: "HDMI Connector"
- note added: "JTAG Debug Port"
- note added: "Overview: Zynq7000 Development Board"
- note added: "PL Configuration"
- note added: "PMIC"
- note added: "PS Configuration"
- note added: "PS MIO Pins"
- note added: "Power Tree Power Sequence"
- note added: "RJ45 Connector"
- note added: "SD Card"
- note added: "SD Card QSPI Flash"
- note added: "SoC Power Pins"
- note added: "To other IC"
- note added: "USB 2.0 Type C"
- note added: "USB High-Spped PHY"
- note added: "USB Type C Power Only"
- note added: "XC7Z010-1CLG400C SoC"
- moved on the sheet: H1, H2, H3, H4

Commit message: update
Other:
- note added: "Power Sequence"
- note added: "USB High-Speed PHY"
- note removed: "Power Tree Power Sequence"
- note removed: "USB High-Spped PHY"
- moved on the sheet: H1, H2, H3, H4
